File: b0_comp.brd (EAGLE design)
At the start: 93 x 70 mm, 1 part

Commit message: .
Parts:
- added C101: 4m7, rcl:E2-5
- added C102: 100n, rcl:C0805
- added IC1: КР1016ВИ1(NE555), st-microelectronics:DIL-08
- added R101*, R101*1: 22k, rcl:M0805
- added R102*: 180k, rcl:M0805
- added R103: 2k2, rcl:M0805
- added VT1: (no value), m_transistor:DPACK
- turned JP1 to 180 degrees
Connections:
- new net +12V: VT1.D
- new net GND: R101*1.1
- new net N$1: JP1.19, JP1.20
- new net N$4: IC1.7, R101*.1, R102*.2
- new net N$5: C101.+, IC1.2, IC1.6, R102*.1
- new net N$6: C102.1, IC1.5
- new net N$7: IC1.3, R103.1
- new net N$8: R103.2, VT1.G
- new net VCC/2: IC1.4, IC1.8, R101*.2
- new net VSS: C101.-, C102.2, IC1.1, R101*1.2, VT1.S
Routing:
- net N$3: track 0.00 -> 4.00 mm
- net N$2: track 0.00 -> 4.00 mm
Changed lines of the file:
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@@
 <setting verticaltext="up"/>
 </settings>
-<grid distance="9.84251969" unitdist="mil" unit="mil" style="lines" multiple="1" display="yes" altdistance="0.025" altunitdist="inch" altunit="inch"/>
+<grid distance="25" unitdist="mil" unit="mil" style="lines" multiple="1" display="yes" altdistance="0.025" altunitdist="inch" altunit="inch"/>
 <layers>
 <layer number="1" name="Top" color="4" fill="1" visible="yes" active="yes"/>
@@
 <layer number="56" name="wert" color="7" fill="1" visible="no" active="no"/>
 <layer number="57" name="tCAD" color="7" fill="1" visible="no" active="no"/>
+<layer number="90" name="Modules" color="7" fill="1" visible="yes" active="yes"/>
 <layer number="91" name="Nets" color="2" fill="1" visible="no" active="no"/>
 <layer number="92" name="Busses" color="1" fill="1" visible="no" active="no"/>
@@
 <layer number="112" name="tSilk" color="7" fill="1" visible="no" active="yes"/>
 <layer number="113" name="ReferenceLS" color="7" fill="1" visible="no" active="no"/>
+<layer number="114" name="bJumper" color="7" fill="1" visible="yes" active="yes"/>
+<layer number="115" name="GND" color="7" fill="1" visible="yes" active="yes"/>
 <layer number="116" name="Patch_BOT" color="9" fill="4" visible="no" active="yes"/>
+<layer number="117" name="tJumper" color="7" fill="1" visible="yes" active="yes"/>
 <layer number="118" name="Rect_Pads" color="7" fill="1" visible="no" active="no"/>
 <layer number="121" name="_tsilk" color="7" fill="1" visible="no" active="yes"/>
@@
 <layer number="251" name="SMDround" color="7" fill="1" visible="no" active="no"/>
 <layer number="254" name="cooling" color="7" fill="1" visible="no" active="yes"/>
+<layer number="255" name="routoute" color="7" fill="1" visible="yes" active="yes"/>
 </layers>
 <board>
@@
 </autorouter>
 <elements>
-<element name="JP1" library="Разъёмы штырьковые 2.54мм" package="1X20" value="" x="-8.371840625" y="-32.50438125"/>
+<element name="JP1" library="Разъёмы штырьковые 2.54мм" package="1X20" value="" x="-8.37" y="-32.5" rot="R180"/>
+<element name="IC1" library="st-microelectronics" package="DIL-08" value="КР1016ВИ1(NE555)" x="60.185" y="30.765">
+<attribute name="OC_NEWARK" value="89K1486" x="60.185" y="30.765" size="1.778" layer="27" display="off"/>
+<attribute name="MPN" value="NE555N" x="60.185" y="30.765" size="1.778" layer="27" display="off"/>
+<attribute name="MF" value="Arrow Electronics" x="60.185" y="30.765" size="1.778" layer="27" display="off"/>
+<attribute name="OC_FARNELL" value="1467742" x="60.185" y="30.765" size="1.778" layer="27" display="off"/>
+</element>
+<element name="R102*" library="rcl" package="M0805" value="180k" x="60.275" y="32.185" rot="MR0"/>
+<element name="R101*" library="rcl" package="M0805" value="22k" x="56.865" y="31.065" rot="MR270"/>
+<element name="C101" library="rcl" package="E2-5" value="4m7" x="57.47" y="24.13" rot="R180"/>
+<element name="C102" library="rcl" package="C0805" value="100n" x="54.26" y="34.24" rot="MR270"/>
+<element name="R103" library="rcl" package="M0805" value="2k2" x="61.395" y="23.445" rot="MR270"/>
+<element name="VT1" library="m_transistor" package="DPACK" value="" x="69.19" y="21.16" rot="MR270"/>
+<element name="R101*1" library="rcl" package="M0805" value="22k" x="58.3" y="19.735" rot="MR0"/>
 </elements>
 <signals>
+<signal name="N$2">
+<wire x1="0" y1="2" x2="0" y2="-2" width="0.1524" layer="1"/>
+</signal>
+<signal name="N$3">
+<wire x1="-2" y1="0" x2="2" y2="0" width="0.1524" layer="1"/>
+</signal>
+<signal name="N$1">
+<contactref element="JP1" pad="20"/>
+<contactref element="JP1" pad="19"/>
+<wire x1="-29.96" y1="-32.5" x2="-32.5" y2="-32.5" width="0" layer="19" extent="1-1"/>
+</signal>
+<signal name="N$5">
+<contactref element="IC1" pad="2"/>
+<contactref element="IC1" pad="6"/>
+<contactref element="R102*" pad="1"/>
+<contactref element="C101" pad="+"/>
+<wire x1="61.225" y1="32.185" x2="61.455" y2="34.575" width="0" layer="19" extent="16-16"/>
+<wire x1="58.915" y1="26.955" x2="61.225" y2="32.185" width="0" layer="19" extent="16-16"/>
+<wire x1="58.486" y1="24.13" x2="58.915" y2="26.955" width="0" layer="19" extent="1-1"/>
+</signal>
+<signal name="N$4">
+<contactref element="R102*" pad="2"/>
+<contactref element="IC1" pad="7"/>
+<contactref element="R101*" pad="1"/>
+<wire x1="59.325" y1="32.185" x2="58.915" y2="34.575" width="0" layer="19" extent="16-16"/>
+<wire x1="56.865" y1="32.015" x2="59.325" y2="32.185" width="0" layer="19" extent="16-16"/>
+</signal>
+<signal name="N$6">
+<contactref element="IC1" pad="5"/>
+<contactref element="C102" pad="1"/>
+<wire x1="54.26" y1="35.19" x2="63.995" y2="34.575" width="0" layer="19" extent="16-16"/>
+</signal>
+<signal name="N$7">
+<contactref element="IC1" pad="3"/>
+<contactref element="R103" pad="1"/>
+<wire x1="61.395" y1="24.395" x2="61.455" y2="26.955" width="0" layer="19" extent="16-16"/>
+</signal>
+<signal name="N$8">
+<contactref element="R103" pad="2"/>
+<contactref element="VT1" pad="G"/>
+<wire x1="61.395" y1="22.495" x2="73.99" y2="23.44" width="0" layer="19" extent="16-16"/>
+</signal>
+<signal name="GND">
+<contactref element="R101*1" pad="1"/>
+</signal>
+<signal name="+12V">
+<contactref element="VT1" pad="D"/>
+</signal>
+<signal name="VSS">
+<contactref element="IC1" pad="1"/>
+<contactref element="C101" pad="-"/>
+<contactref element="C102" pad="2"/>
+<contactref element="VT1" pad="S"/>
+<contactref element="R101*1" pad="2"/>
+<wire x1="56.375" y1="26.955" x2="54.26" y2="33.29" width="0" layer="19" extent="16-16"/>
+<wire x1="56.454" y1="24.13" x2="56.375" y2="26.955" width="0" layer="19" extent="1-1"/>
+<wire x1="57.35" y1="19.735" x2="56.454" y2="24.13" width="0" layer="19" extent="16-16"/>
+<wire x1="73.99" y1="18.88" x2="57.35" y2="19.735" width="0" layer="19" extent="16-16"/>
+</signal>
+<signal name="VCC/2">
+<contactref element="IC1" pad="4"/>
+<contactref element="IC1" pad="8"/>
+<contactref element="R101*" pad="2"/>
+<wire x1="56.865" y1="30.115" x2="63.995" y2="26.955" width="0" layer="19" extent="16-16"/>
+<wire x1="56.375" y1="34.575" x2="56.865" y2="30.115" width="0" layer="19" extent="16-16"/>
+</signal>
 </signals>
 </board>

Commit message: .
Parts:
- added IC2: UC3843N, v-reg:DIL08
- added IC3: MEGA8-AI, atmel:TQFP32-08
- added JP2, JP3, JP4, JP5: (no value), Разъёмы штырьковые 2.54мм:1X01
- added U$1: GD75232DB, GD75232:SSOP20D8
Connections:
- removed net VCC/2: IC1.4, IC1.8, R101*.2
- removed net VSS: C101.-, C102.2, IC1.1, R101*1.2, VT1.S
- new net +5V: U$1.20
- new net -12V: U$1.10
- new net AVCC: IC3.18
- new net N$10: C101.-, C102.2, IC1.1, JP3.1, R101*1.2, VT1.S
- new net N$9: IC1.4, IC1.8, JP2.1, R101*.2
- new net VCC: IC2.7, IC3.4, IC3.6
- net +12V: now also JP4.1, U$1.1
- net GND: now also IC2.5, IC3.21, IC3.3, IC3.5, JP5.1, U$1.11
Changed lines of the file:
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@@
 <element name="VT1" library="m_transistor" package="DPACK" value="" x="69.19" y="21.16" rot="MR270"/>
 <element name="R101*1" library="rcl" package="M0805" value="22k" x="58.3" y="19.735" rot="MR0"/>
+<element name="JP2" library="Разъёмы штырьковые 2.54мм" package="1X01" value="" x="78.74" y="27.305"/>
+<element name="JP3" library="Разъёмы штырьковые 2.54мм" package="1X01" value="" x="78.74" y="15.24"/>
+<element name="JP4" library="Разъёмы штырьковые 2.54мм" package="1X01" value="" x="79.375" y="21.59"/>
+<element name="JP5" library="Разъёмы штырьковые 2.54мм" package="1X01" value="" x="59.69" y="13.335"/>
+<element name="IC2" library="v-reg" package="DIL08" value="UC3843N" x="74.295" y="-10.795"/>
+<element name="IC3" library="atmel" package="TQFP32-08" value="MEGA8-AI" x="-7.62" y="-50.8" rot="MR0">
+<attribute name="OC_NEWARK" value="73M8863" x="-7.62" y="-50.8" size="1.778" layer="28" rot="MR0" display="off"/>
+<attribute name="MPN" value="ATMEGA8-16AU" x="-7.62" y="-50.8" size="1.778" layer="28" rot="MR0" display="off"/>
+<attribute name="MF" value="" x="-7.62" y="-50.8" size="1.778" layer="28" rot="MR0" display="off"/>
+<attribute name="OC_FARNELL" value="9171371" x="-7.62" y="-50.8" size="1.778" layer="28" rot="MR0" display="off"/>
+</element>
+<element name="U$1" library="GD75232" package="SSOP20D8" value="GD75232DB" x="-11.43" y="-63.5" rot="MR0"/>
 </elements>
 <signals>
@@
 <signal name="GND">
 <contactref element="R101*1" pad="1"/>
+<contactref element="JP5" pad="1"/>
+<contactref element="IC2" pad="5"/>
+<contactref element="IC3" pad="3"/>
+<contactref element="IC3" pad="5"/>
+<contactref element="IC3" pad="21"/>
+<contactref element="U$1" pad="11"/>
+<wire x1="-11.9126" y1="-50.4" x2="-14.351" y2="-60.2488" width="0" layer="19" extent="16-16"/>
+<wire x1="-3.3274" y1="-51.2" x2="-11.9126" y2="-50.4" width="0" layer="19" extent="16-16"/>
+<wire x1="-3.3274" y1="-49.6" x2="-3.3274" y2="-51.2" width="0" layer="19" extent="16-16"/>
+<wire x1="59.69" y1="13.335" x2="-3.3274" y2="-49.6" width="0" layer="19" extent="16-16"/>
+<wire x1="59.25" y1="19.735" x2="59.69" y2="13.335" width="0" layer="19" extent="16-16"/>
+<wire x1="78.105" y1="-6.985" x2="59.69" y2="13.335" width="0" layer="19" extent="1-1"/>
 </signal>
 <signal name="+12V">
 <contactref element="VT1" pad="D"/>
+<contactref element="JP4" pad="1"/>
+<contactref element="U$1" pad="1"/>
+<wire x1="66.69" y1="21.16" x2="79.375" y2="21.59" width="0" layer="19" extent="16-16"/>
+<wire x1="-8.636" y1="-66.8528" x2="66.69" y2="21.16" width="0" layer="19" extent="16-16"/>
 </signal>
-<signal name="VSS">
+<signal name="N$9">
+<contactref element="IC1" pad="4"/>
+<contactref element="IC1" pad="8"/>
+<contactref element="R101*" pad="2"/>
+<contactref element="JP2" pad="1"/>
+<wire x1="63.995" y1="26.955" x2="78.74" y2="27.305" width="0" layer="19" extent="1-1"/>
+<wire x1="56.865" y1="30.115" x2="63.995" y2="26.955" width="0" layer="19" extent="16-16"/>
+<wire x1="56.375" y1="34.575" x2="56.865" y2="30.115" width="0" layer="19" extent="16-16"/>
+</signal>
+<signal name="N$10">
 <contactref element="IC1" pad="1"/>
 <contactref element="C101" pad="-"/>
@@
 <contactref element="VT1" pad="S"/>
 <contactref element="R101*1" pad="2"/>
-<wire x1="56.375" y1="26.955" x2="54.26" y2="33.29" width="0" layer="19" extent="16-16"/>
-<wire x1="56.454" y1="24.13" x2="56.375" y2="26.955" width="0" layer="19" extent="1-1"/>
-<wire x1="57.35" y1="19.735" x2="56.454" y2="24.13" width="0" layer="19" extent="16-16"/>
-<wire x1="73.99" y1="18.88" x2="57.35" y2="19.735" width="0" layer="19" extent="16-16"/>
+<contactref element="JP3" pad="1"/>
+<wire x1="73.99" y1="18.88" x2="78.74" y2="15.24" width="0" layer="19" extent="16-16"/>
+<wire x1="57.35" y1="19.735" x2="73.99" y2="18.88" width="0" layer="19" extent="16-16"/>
+<wire x1="56.454" y1="24.13" x2="57.35" y2="19.735" width="0" layer="19" extent="16-16"/>
+<wire x1="56.375" y1="26.955" x2="56.454" y2="24.13" width="0" layer="19" extent="1-1"/>
+<wire x1="54.26" y1="33.29" x2="56.375" y2="26.955" width="0" layer="19" extent="16-16"/>
 </signal>
-<signal name="VCC/2">
-<contactref element="IC1" pad="4"/>
-<contactref element="IC1" pad="8"/>
-<contactref element="R101*" pad="2"/>
-<wire x1="56.865" y1="30.115" x2="63.995" y2="26.955" width="0" layer="19" extent="16-16"/>
-<wire x1="56.375" y1="34.575" x2="56.865" y2="30.115" width="0" layer="19" extent="16-16"/>
+<signal name="VCC">
+<contactref element="IC2" pad="7"/>
+<contactref element="IC3" pad="4"/>
+<contactref element="IC3" pad="6"/>
+<wire x1="-3.3274" y1="-50.4" x2="73.025" y2="-6.985" width="0" layer="19" extent="16-16"/>
+<wire x1="-3.3274" y1="-52" x2="-3.3274" y2="-50.4" width="0" layer="19" extent="16-16"/>
+</signal>
+<signal name="AVCC">
+<contactref element="IC3" pad="18"/>
+</signal>
+<signal name="-12V">
+<contactref element="U$1" pad="10"/>
+</signal>
+<signal name="+5V">
+<contactref element="U$1" pad="20"/>
 </signal>
 </signals>

Commit message: .
Parts:
- added C1, C2, C3: 1n, rcl:C0805
- added C4: 100n, rcl:C0805
- added IC4, IC5: MEGA16-P, atmel:DIL40
- added IC6: MEGA8-P, atmel:DIL28-3
- added R1: 4r7, rcl:M0805
- added R2: 330, rcl:M0805
- added R3: 0e1 2w, rcl:M0805
- added R4: 15k, rcl:M0805
- added R5: 100k, rcl:M0805
- added R6: 10r, rcl:M0805
- added VT2: (no value), m_transistor:DPACK
- moved IC2 114.7 mm to (-38.1, 12.1)
- moved U$1 80.7 mm to (18.4, 11.4), turned to 270 degrees
- moved IC3 36.8 mm to (-17.1, -15.2)
Connections:
- new net N$11: IC5.35, IC6.28
- new net N$12: IC5.36, IC6.27
- new net N$13: IC5.37, IC6.26
- new net N$14: IC5.38, IC6.25
- new net N$15: IC5.39, IC6.24
- new net N$16: IC5.40, IC6.23
- new net N$17: IC5.6, IC6.17
- new net N$18: IC5.7, IC6.18
- new net N$19: IC5.8, IC6.19
- new net N$20: IC2.6, R1.1
- new net N$21: R1.2, VT2.G
- new net N$22: C2.1, IC2.3, R2.1
- new net N$23: R2.2, R3.2, VT2.S
- new net N$24: VT2.D
- new net N$25: IC2.8, R4.2
- new net N$26: C1.1, IC2.4, R4.1
- new net N$28: C3.2, IC2.2, R5.1
- new net N$29: C3.1, IC2.1, R5.2
- new net N$30: C4.2, IC2.7, R6.1
- net +12V: now also R6.2
- net AVCC: now also IC4.30, IC5.30, IC6.20
- net GND: now also C1.2, C2.2, C4.1, IC4.11, IC4.31, IC5.11, IC5.31, IC6.22, IC6.8, R3.1
- net VCC: now also IC4.10, IC5.10, IC6.7; no longer IC2.7

Commit message: .
Parts:
- IC6: value MEGA8-P -> MEGA8-AI; device atmel:DIL28-3 -> atmel:TQFP32-08
- moved IC5 8.47 mm to (-26.0, -65.4)
- moved VT2 7.75 mm to (-27.9, 29.2)
- moved IC6 2.84 mm to (-37.5, -64.8), flipped to the bottom, turned to 15 degrees
Connections:
- new net N$27: IC5.6, IC6.12
- new net N$31: IC5.7, IC6.11
- new net N$32: IC5.8, IC6.10
- new net N$33: IC5.32, IC6.20
- new net N$34: IC5.30, IC6.18
- new net N$35: IC5.34, IC6.27
- new net N$36: IC5.35, IC6.26
- new net N$37: IC5.36, IC6.25
- new net N$38: IC5.37, IC6.24
- new net N$39: IC5.33, IC6.28
- new net N$40: IC5.38, IC6.23
- new net N$41: IC5.40, IC6.19
- new net N$42: IC5.39, IC6.22
- new net N$43: IC5.27, IC6.32
- new net N$44: IC5.9, IC6.29
- new net N$45: IC5.29, IC6.30
- new net N$46: IC5.28, IC6.31
- new net N$47: IC5.26, IC6.1
- new net N$48: IC5.25, IC6.2
- new net N$49: IC5.24, IC6.9
- net AVCC: no longer IC5.30, IC6.20
- net GND: no longer IC5.11, IC5.31, IC6.22, IC6.8
- net N$11: now also IC5.13, IC6.7; no longer IC5.35, IC6.28
- net N$12: now also IC5.12, IC6.8; no longer IC5.36, IC6.27
- net N$13: now also IC5.11, IC5.31, IC6.21, IC6.3, IC6.5; no longer IC5.37, IC6.26
- net N$14: now also IC5.1, IC6.17; no longer IC5.38, IC6.25
- net N$15: now also IC5.10, IC6.4, IC6.6; no longer IC5.39, IC6.24
- net N$16: now also IC5.2, IC6.16; no longer IC5.40, IC6.23
- net N$17: now also IC5.3, IC6.15; no longer IC5.6, IC6.17
- net N$18: now also IC5.4, IC6.14; no longer IC5.7, IC6.18
- net N$19: now also IC5.5, IC6.13; no longer IC5.8, IC6.19
- net VCC: no longer IC5.10, IC6.7
Routing:
- net N$48: track 0.00 -> 24.9 mm
- net N$49: track 0.00 -> 23.7 mm
- net N$47: track 0.00 -> 21.8 mm
- net N$33: track 0.00 -> 21.4 mm, vias 0 -> 2
- net N$43: track 0.00 -> 19.3 mm
- net N$44: track 0.00 -> 19.0 mm, vias 0 -> 2
- net N$46: track 0.00 -> 17.0 mm
- net N$45: track 0.00 -> 15.6 mm
- net N$34: track 0.00 -> 12.4 mm
Other:
- board text added: "m-16-aref"
- board text added: "m-16-gnd"
- board text added: "m-16-vcc"
- board text added: "m-16-xtal1"
- board text added: "m-16-xtal2"
- board text added: "m16-0"
- board text added: "m16-1"
- board text added: "m16-10"
- board text added: "m16-11"
- board text added: "m16-12"
- board text added: "m16-13"
- board text added: "m16-14"
- board text added: "m16-15"
- board text added: "m16-16"
- board text added: "m16-17"
- board text added: "m16-18"
- board text added: "m16-19"
- board text added: "m16-2"
- board text added: "m16-20"
- board text added: "m16-21"
- board text added: "m16-22"
- board text added: "m16-23"
- board text added: "m16-3"
- board text added: "m16-4"
- board text added: "m16-5"
- board text added: "m16-6"
- board text added: "m16-7"
- board text added: "m16-8"
- board text added: "m16-9"
- board text added: "m16-a0"
- board text added: "m16-a1"
- board text added: "m16-a2"
- board text added: "m16-a3"
- board text added: "m16-a4"
- board text added: "m16-a5"
- board text added: "m16-a6"
- board text added: "m16-a7"
- board text added: "m16-avcc"
- board text added: "m8-10"
- board text added: "m8-11-mosi"
- board text added: "m8-12-miso"
- board text added: "m8-13-sck"
- board text added: "m8-6"
- board text added: "m8-7"
- board text added: "m8-8"
- board text added: "m8-9"
- board text added: "m8-a0"
- board text added: "m8-a1"
- board text added: "m8-a2"
- board text added: "m8-a3"
- board text added: "m8-a4"
- board text added: "m8-a5"
- board text added: "m8-adc6"
- board text added: "m8-adc7"
- board text added: "reset"

Commit message: .
Parts:
- moved IC6 0.90 mm to (-38.1, -65.4), turned to 5 degrees
Routing:
- net N$13: track 0.00 -> 29.7 mm, vias 0 -> 1
- net N$34: track 12.4 -> 41.6 mm, vias 0 -> 2
- net N$11: track 0.00 -> 19.4 mm
- net N$12: track 0.00 -> 17.0 mm
- net N$15: track 0.00 -> 16.3 mm, vias 0 -> 2
- net N$41: track 0.00 -> 13.4 mm
- net N$14: track 0.00 -> 10.8 mm
- net N$42: track 0.00 -> 9.35 mm
- net N$16: track 0.00 -> 8.96 mm
- net N$49: track 23.7 -> 32.4 mm, vias 0 -> 2
- net N$17: track 0.00 -> 7.29 mm
- net N$33: track 21.4 -> 28.5 mm
- net N$40: track 0.00 -> 6.92 mm
- net N$32: track 0.00 -> 5.98 mm
- net N$18: track 0.00 -> 5.38 mm
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
Commit message: .
Parts:
- added C5: (no value), rcl:C0805
- added JP6: (no value), Разъёмы штырьковые 2.54мм:1X20
- IC5: device atmel:DIL40 -> b0ic:DIL40
- moved IC6 1.42 mm to (-36.8, -66.0), turned to 10 degrees
Connections:
- net N$1: now also JP6.19, JP6.20
- net N$13: now also C5.1
- net N$15: now also C5.2
Routing:
- net N$13: track 29.7 -> 37.7 mm, vias 1 -> 2
- net N$39: track 0.00 -> 6.58 mm
- net N$34: track 41.6 -> 36.8 mm
- net N$35: track 0.00 -> 4.79 mm
- net N$37: track 0.00 -> 4.02 mm
- net N$36: track 0.00 -> 3.92 mm
- net N$15: track 16.3 -> 13.6 mm
- net N$41: track 13.4 -> 15.4 mm
- net N$38: track 4.63 -> 6.14 mm
- net N$40: track 6.92 -> 8.43 mm
- net N$33: track 28.5 -> 27.1 mm
- net N$42: track 9.35 -> 10.8 mm
- net N$45: track 16.6 -> 17.8 mm
- net N$44: track 23.3 -> 24.6 mm
- net N$11: track 19.4 -> 18.2 mm
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
Commit message: .
Parts:
- added SJ1, SJ2, SJ3, SJ4, SJ5, SJ6, SJ7, SJ8: (no value), jumper:SJ
- moved JP6 0.32 mm to (-8.57, -28.3), turned to 180 degrees
Connections:
- new net N$50: IC5.33, SJ1.1
- new net N$51: IC5.35, SJ3.1
- new net N$52: IC5.37, SJ5.1
- new net N$53: IC5.39, SJ7.1
- new net N$54: IC5.40, SJ8.1
- new net N$55: IC5.38, SJ6.1
- new net N$56: IC5.36, SJ4.1
- new net N$57: IC5.34, SJ2.1
- net N$35: now also SJ2.2; no longer IC5.34
- net N$36: now also SJ3.2; no longer IC5.35
- net N$37: now also SJ4.2; no longer IC5.36
- net N$38: now also SJ5.2; no longer IC5.37
- net N$39: now also SJ1.2; no longer IC5.33
- net N$40: now also SJ6.2; no longer IC5.38
- net N$41: now also SJ8.2; no longer IC5.40
- net N$42: now also SJ7.2; no longer IC5.39
Routing:
- net N$39: track 6.58 -> 0.00 mm
- net N$41: track 15.4 -> 9.95 mm
- net N$35: track 4.79 -> 0.00 mm
- net N$38: track 6.14 -> 2.10 mm
- net N$37: track 4.02 -> 0.00 mm
- net N$36: track 3.92 -> 0.00 mm
- net N$42: track 10.8 -> 7.49 mm
- net N$40: track 8.43 -> 6.60 mm
- net N$33: track 27.1 -> 28.3 mm

Commit message: .
Parts:
- added M1: ARDUINO-PRO-MINI-5.0V, diy-modules:ARDUINO-PRO-MINI
- added M2: ARDUINO-NANO-3.0#ISP, diy-modules:ARDUINO-NANO-3.0#ISP
Connections:
- new net 3V3: M2.J2.14
- new net 5V: M2.J2.4
- new net GND.1: M1.J7.9
- new net GND.2: M1.J6.2, M2.J2.2
- new net N$58: M1.J7.12, M2.J1.1
- new net N$59: M1.J7.11, M2.J1.2
- new net N$60: M1.J7.10, M2.J1.3
- new net N$61: M2.J1.4
- new net RAW: M1.J6.1
- new net VIN: M2.J2.1
- net VCC: now also M1.J6.4
Changed lines of the file:
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@@
 <element name="SJ7" library="jumper" package="SJ" value="" x="-47.625" y="-60.325" rot="MR270"/>
 <element name="SJ8" library="jumper" package="SJ" value="" x="-50.165" y="-60.325" rot="MR270"/>
+<element name="M1" library="diy-modules" package="ARDUINO-PRO-MINI" value="ARDUINO-PRO-MINI-5.0V" x="24.765" y="-73.3425"/>
+<element name="M2" library="diy-modules" package="ARDUINO-NANO-3.0#ISP" value="ARDUINO-NANO-3.0#ISP" x="44.7675" y="-48.5775" rot="R180"/>
 </elements>
 <signals>
@@
 <contactref element="IC3" pad="6"/>
 <contactref element="IC4" pad="10"/>
+<contactref element="M1" pad="J6.4"/>
+<wire x1="-16.51" y1="-22.225" x2="19.685" y2="-65.7225" width="0" layer="19" extent="1-1"/>
 <wire x1="-12.8524" y1="-16.44" x2="-16.51" y2="-22.225" width="0" layer="19" extent="16-16"/>
 <wire x1="-12.8524" y1="-14.84" x2="-12.8524" y2="-16.44" width="0" layer="19" extent="16-16"/>
@@
 <wire x1="-34.925" y1="-57.9755" x2="-34.925" y2="-57.785" width="0" layer="19" extent="16-16"/>
 </signal>
+<signal name="GND.1">
+<contactref element="M1" pad="J7.9"/>
+</signal>
+<signal name="RAW">
+<contactref element="M1" pad="J6.1"/>
+</signal>
+<signal name="GND.2">
+<contactref element="M1" pad="J6.2"/>
+<contactref element="M2" pad="J2.2"/>
+<wire x1="14.605" y1="-65.7225" x2="29.5275" y2="-40.9575" width="0" layer="19" extent="1-1"/>
+</signal>
+<signal name="VIN">
+<contactref element="M2" pad="J2.1"/>
+</signal>
+<signal name="5V">
+<contactref element="M2" pad="J2.4"/>
+</signal>
+<signal name="3V3">
+<contactref element="M2" pad="J2.14"/>
+</signal>
+<signal name="N$58">
+<contactref element="M1" pad="J7.12"/>
+<contactref element="M2" pad="J1.1"/>
+<wire x1="26.9875" y1="-56.1975" x2="12.065" y2="-80.9625" width="0" layer="19" extent="1-1"/>
+</signal>
+<signal name="N$59">
+<contactref element="M1" pad="J7.11"/>
+<contactref element="M2" pad="J1.2"/>
+<wire x1="29.5275" y1="-56.1975" x2="14.605" y2="-80.9625" width="0" layer="19" extent="1-1"/>
+</signal>
+<signal name="N$60">
+<contactref element="M1" pad="J7.10"/>
+<contactref element="M2" pad="J1.3"/>
+<wire x1="32.0675" y1="-56.1975" x2="17.145" y2="-80.9625" width="0" layer="19" extent="1-1"/>
+</signal>
+<signal name="N$61">
+<contactref element="M2" pad="J1.4"/>
+</signal>
 </signals>
