File: b0_comp.brd (EAGLE design)
At the start: 93 x 70 mm, 282 parts, among them IC1 КР1006ВИ1(NE555), IC3 LM358D, IC4 78L09F, IC6 MEGA8-AI, IC7 74121N, IC8 4030N, IC9 LM324D, T1P T90, -26 MicroMetals Yellow-W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

Commit message: .
Parts:
- added C2: (no value), rcl:E2,5-5
- added IC5: XL6009S, XL6009:TO263-5
- added R8P1: 8k6, rcl:M0805
- added R8P2: 1k, rcl:M0805
- added VD2P1: SR5200, diode:CB429-17
- moved DA5 319.7 mm to (-300.4, 119.4)
- moved DA6 319.7 mm to (-284.5, 118.7)
- moved R20 319.7 mm to (-297.8, 119.4)
- moved R21 319.7 mm to (-294.6, 120.7)
- moved R22 319.7 mm to (-275.6, 114.3)
- moved R23 319.7 mm to (-276.2, 123.2)
- moved R3 319.7 mm to (-300.4, 119.4)
Connections:
- new net N$185: C2.+, IC5.3
- new net N$186: IC5.4
- new net N$187: R8P1.2, VD2P1.C
- new net N$188: C2.-, VD2P1.A
- new net N$189: IC5.5, R8P1.1, R8P2.2
- net GND: now also IC5.1, IC5.2, R8P2.1

Commit message: .
Parts:
- added R8P3: 3k, rcl:M0805
- added T1P1: T90, -26 MicroMetals Yellow-White, b0f:R23X14
- added VD2P2: SR5200, diode:CB429-17
- C2: value (none) -> 22m
- IC5: value XL6009S -> XL6009
- moved C2 7.10 mm to (-367.7, 91.4)
- moved VD2P1 4.02 mm to (-360.0, 90.8)
- moved R8P1 2.01 mm to (-370.8, 79.4)
- moved R8P2 1.90 mm to (-379.7, 83.8)
Connections:
- new net N$190: C2.-, VD2P2.A
- new net N$191: VD2P2.C
- net N$187: now also R8P3.2; no longer R8P1.2
- net N$188: no longer C2.-
- net N$189: now also R8P3.1; no longer R8P1.1
Changed lines of the file:
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@@
 <element name="R22" library="rcl" package="M0805" value="27" x="-275.59" y="114.3" rot="MR180"/>
 <element name="R23" library="rcl" package="M0805" value="27" x="-276.225" y="123.19" rot="MR180"/>
-<element name="IC5" library="XL6009" package="TO263-5" value="XL6009S" x="-376.555" y="95.25"/>
-<element name="VD2P1" library="diode" package="CB429-17" value="SR5200" x="-361.315" y="86.995" rot="R90"/>
-<element name="C2" library="rcl" package="E2,5-5" value="" x="-368.935" y="84.455"/>
-<element name="R8P1" library="rcl" package="M0805" value="8k6" x="-371.475" y="77.47"/>
-<element name="R8P2" library="rcl" package="M0805" value="1k" x="-379.73" y="81.915"/>
+<element name="IC5" library="XL6009" package="TO263-5" value="XL6009" x="-376.555" y="95.25"/>
+<element name="VD2P1" library="diode" package="CB429-17" value="SR5200" x="-360.045" y="90.805" rot="R90"/>
+<element name="C2" library="rcl" package="E2,5-5" value="22m" x="-367.665" y="91.44"/>
+<element name="R8P1" library="rcl" package="M0805" value="8k6" x="-370.84" y="79.375"/>
+<element name="R8P2" library="rcl" package="M0805" value="1k" x="-379.73" y="83.82"/>
+<element name="R8P3" library="rcl" package="M0805" value="3k" x="-371.475" y="83.82"/>
+<element name="T1P1" library="b0f" package="R23X14" value="T90, -26 MicroMetals Yellow-White" x="-370.205" y="117.475"/>
+<element name="VD2P2" library="diode" package="CB429-17" value="SR5200" x="-353.695" y="88.9" rot="R90"/>
 </elements>
 <signals>
@@
 <wire x1="-367.0275" y1="-35.2425" x2="-364.4265" y2="-29.5275" width="0" layer="19" extent="1-1"/>
 <wire x1="-364.4265" y1="-39.0525" x2="-367.0275" y2="-35.2425" width="0" layer="19" extent="1-1"/>
-<wire x1="-380.68" y1="81.915" x2="-367.3475" y2="-3.4925" width="0" layer="19" extent="1-1"/>
-<wire x1="-379.9586" y1="89.4588" x2="-380.68" y2="81.915" width="0" layer="19" extent="1-1"/>
+<wire x1="-380.68" y1="83.82" x2="-367.3475" y2="-3.4925" width="0" layer="19" extent="1-1"/>
+<wire x1="-379.9586" y1="89.4588" x2="-380.68" y2="83.82" width="0" layer="19" extent="1-1"/>
 <wire x1="-378.2568" y1="89.4588" x2="-379.9586" y2="89.4588" width="0" layer="19" extent="1-1"/>
 </signal>
@@
 <contactref element="IC5" pad="3"/>
 <contactref element="C2" pad="+"/>
-<wire x1="-370.205" y1="84.455" x2="-376.555" y2="89.4588" width="0" layer="19" extent="1-1"/>
+<wire x1="-368.935" y1="91.44" x2="-376.555" y2="89.4588" width="0" layer="19" extent="1-1"/>
 </signal>
 <signal name="N$186">
@@
 <signal name="N$188">
 <contactref element="VD2P1" pad="A"/>
-<contactref element="C2" pad="-"/>
-<wire x1="-361.315" y1="95.885" x2="-367.665" y2="84.455" width="0" layer="19" extent="1-1"/>
 </signal>
 <signal name="N$187">
 <contactref element="VD2P1" pad="C"/>
-<contactref element="R8P1" pad="2"/>
-<wire x1="-361.315" y1="78.105" x2="-370.525" y2="77.47" width="0" layer="19" extent="1-1"/>
+<contactref element="R8P3" pad="2"/>
+<wire x1="-370.525" y1="83.82" x2="-360.045" y2="81.915" width="0" layer="19" extent="1-1"/>
 </signal>
 <signal name="N$189">
-<contactref element="R8P1" pad="1"/>
 <contactref element="R8P2" pad="2"/>
 <contactref element="IC5" pad="5"/>
-<wire x1="-372.425" y1="77.47" x2="-378.78" y2="81.915" width="0" layer="19" extent="1-1"/>
-<wire x1="-373.1514" y1="89.4588" x2="-378.78" y2="81.915" width="0" layer="19" extent="1-1"/>
+<contactref element="R8P3" pad="1"/>
+<wire x1="-373.1514" y1="89.4588" x2="-378.78" y2="83.82" width="0" layer="19" extent="1-1"/>
+<wire x1="-372.425" y1="83.82" x2="-378.78" y2="83.82" width="0" layer="19" extent="1-1"/>
+</signal>
+<signal name="N$190">
+<contactref element="C2" pad="-"/>
+<contactref element="VD2P2" pad="A"/>
+<wire x1="-353.695" y1="97.79" x2="-366.395" y2="91.44" width="0" layer="19" extent="1-1"/>
+</signal>
+<signal name="N$191">
+<contactref element="VD2P2" pad="C"/>
 </signal>
 </signals>

Commit message: .
Parts:
- moved VD2P2 2.54 mm to (-353.7, 91.4)
- moved C2 1.27 mm to (-367.7, 92.7)
- moved VD2P1 0.90 mm to (-360.7, 91.4)
Changed lines of the file:
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@@
 <element name="R23" library="rcl" package="M0805" value="27" x="-276.225" y="123.19" rot="MR180"/>
 <element name="IC5" library="XL6009" package="TO263-5" value="XL6009" x="-376.555" y="95.25"/>
-<element name="VD2P1" library="diode" package="CB429-17" value="SR5200" x="-360.045" y="90.805" rot="R90"/>
-<element name="C2" library="rcl" package="E2,5-5" value="22m" x="-367.665" y="91.44"/>
+<element name="VD2P1" library="diode" package="CB429-17" value="SR5200" x="-360.68" y="91.44" rot="R90"/>
+<element name="C2" library="rcl" package="E2,5-5" value="22m" x="-367.665" y="92.71"/>
 <element name="R8P1" library="rcl" package="M0805" value="8k6" x="-370.84" y="79.375"/>
 <element name="R8P2" library="rcl" package="M0805" value="1k" x="-379.73" y="83.82"/>
 <element name="R8P3" library="rcl" package="M0805" value="3k" x="-371.475" y="83.82"/>
 <element name="T1P1" library="b0f" package="R23X14" value="T90, -26 MicroMetals Yellow-White" x="-370.205" y="117.475"/>
-<element name="VD2P2" library="diode" package="CB429-17" value="SR5200" x="-353.695" y="88.9" rot="R90"/>
+<element name="VD2P2" library="diode" package="CB429-17" value="SR5200" x="-353.695" y="91.44" rot="R90"/>
 </elements>
 <signals>
@@
 <contactref element="IC5" pad="3"/>
 <contactref element="C2" pad="+"/>
-<wire x1="-368.935" y1="91.44" x2="-376.555" y2="89.4588" width="0" layer="19" extent="1-1"/>
+<wire x1="-368.935" y1="92.71" x2="-376.555" y2="89.4588" width="0" layer="19" extent="1-1"/>
 </signal>
 <signal name="N$186">
@@
 <contactref element="VD2P1" pad="C"/>
 <contactref element="R8P3" pad="2"/>
-<wire x1="-370.525" y1="83.82" x2="-360.045" y2="81.915" width="0" layer="19" extent="1-1"/>
+<wire x1="-370.525" y1="83.82" x2="-360.68" y2="82.55" width="0" layer="19" extent="1-1"/>
 </signal>
 <signal name="N$189">
@@
 <contactref element="C2" pad="-"/>
 <contactref element="VD2P2" pad="A"/>
-<wire x1="-353.695" y1="97.79" x2="-366.395" y2="91.44" width="0" layer="19" extent="1-1"/>
+<wire x1="-353.695" y1="100.33" x2="-366.395" y2="92.71" width="0" layer="19" extent="1-1"/>
 </signal>
 <signal name="N$191">

Commit message: .
Parts:
- removed R8P1: 8k6, rcl:M0805
- added C3: 22m, rcl:E2,5-5
- added Q1: (no value), transistor-fet:P-TO247
- added VD10P1, VD9P1, VD9P3: (no value), diode:CB429-17
- added VD2P3: SR5200, diode:CB429-17
- T1P1: value T90, -26 MicroMetals Yellow-White -> (none)
Connections:
- removed net N$187: R8P3.2, VD2P1.C
- new net N$192: Q1.3
- new net N$193: Q1.2
- new net N$194: Q1.1
- new net N$195: VD2P3.A
- new net N$196: VD10P1.A
- new net N$197: VD9P1.C
- net +12V: now also VD10P1.C
- net +18V: now also VD2P3.C
- net +5VUSB: now also R8P3.2, VD2P1.C
- net +7V5: now also VD2P2.C
- net -12V: now also VD9P3.A
- net -18V: now also VD9P1.A
- net N$185: now also C3.+
- net N$188: now also C2.-, C3.-
- net N$190: no longer C2.-
- net N$191: now also VD9P3.C; no longer VD2P2.C
Changed lines of the file:
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@@
 <element name="VD2P1" library="diode" package="CB429-17" value="SR5200" x="-360.68" y="91.44" rot="R90"/>
 <element name="C2" library="rcl" package="E2,5-5" value="22m" x="-367.665" y="92.71"/>
-<element name="R8P1" library="rcl" package="M0805" value="8k6" x="-370.84" y="79.375"/>
 <element name="R8P2" library="rcl" package="M0805" value="1k" x="-379.73" y="83.82"/>
 <element name="R8P3" library="rcl" package="M0805" value="3k" x="-371.475" y="83.82"/>
-<element name="T1P1" library="b0f" package="R23X14" value="T90, -26 MicroMetals Yellow-White" x="-370.205" y="117.475"/>
+<element name="T1P1" library="b0f" package="R23X14" value="" x="-370.205" y="117.475"/>
 <element name="VD2P2" library="diode" package="CB429-17" value="SR5200" x="-353.695" y="91.44" rot="R90"/>
+<element name="Q1" library="transistor-fet" package="P-TO247" value="" x="-396.24" y="-146.05"/>
+<element name="C3" library="rcl" package="E2,5-5" value="22m" x="-401.32" y="-179.705"/>
+<element name="VD2P3" library="diode" package="CB429-17" value="SR5200" x="-392.43" y="-187.325"/>
+<element name="VD10P1" library="diode" package="CB429-17" value="" x="-392.43" y="-194.945"/>
+<element name="VD9P3" library="diode" package="CB429-17" value="" x="-392.43" y="-217.805"/>
+<element name="VD9P1" library="diode" package="CB429-17" value="" x="-392.43" y="-225.425"/>
 </elements>
 <signals>
@@
 <contactref element="F_MAIN_POWER" pad="14A"/>
 <contactref element="F_MAIN_POWER" pad="14"/>
+<contactref element="VD10P1" pad="C"/>
 <wire x1="-39.95" y1="-29.5" x2="-117.16" y2="-58.42" width="0" layer="19" extent="1-1"/>
 <wire x1="-40.27" y1="-26.31" x2="-39.95" y2="-29.5" width="0" layer="19" extent="1-1"/>
@@
 <wire x1="-365.1275" y1="-14.9225" x2="-362.6075" y2="-24.4475" width="0" layer="19" extent="1-1"/>
 <wire x1="-362.2675" y1="5.3975" x2="-365.1275" y2="-14.9225" width="0" layer="19" extent="1-1"/>
+<wire x1="-401.32" y1="-194.945" x2="-362.6075" y2="-24.4475" width="0" layer="19" extent="1-1"/>
 </signal>
 <signal name="N$9">
@@
 <contactref element="VD8P" pad="A"/>
 <contactref element="19" pad="1"/>
-<wire x1="54.6528" y1="-15.359" x2="127" y2="-62.70625" width="0" layer="19" extent="1-1"/>
-<wire x1="17.78" y1="-76.835" x2="54.6528" y2="-15.359" width="0" layer="19" extent="1-1"/>
+<contactref element="VD9P3" pad="A"/>
+<wire x1="17.78" y1="-76.835" x2="-383.54" y2="-217.805" width="0" layer="19" extent="1-1"/>
+<wire x1="54.6528" y1="-15.359" x2="17.78" y2="-76.835" width="0" layer="19" extent="1-1"/>
+<wire x1="127" y1="-62.70625" x2="54.6528" y2="-15.359" width="0" layer="19" extent="1-1"/>
 </signal>
 <signal name="+5V">
@@
 <contactref element="VD2P" pad="C"/>
 <contactref element="C7P" pad="+"/>
+<contactref element="VD2P1" pad="C"/>
+<contactref element="R8P3" pad="2"/>
 <wire x1="3.175" y1="-93.98" x2="-29.05375" y2="-90.17" width="0" layer="19" extent="1-1"/>
 <wire x1="35.8775" y1="-96.2025" x2="3.175" y2="-93.98" width="0" layer="19" extent="1-1"/>
+<wire x1="-360.68" y1="82.55" x2="-29.05375" y2="-90.17" width="0" layer="19" extent="1-1"/>
+<wire x1="-370.525" y1="83.82" x2="-360.68" y2="82.55" width="0" layer="19" extent="1-1"/>
 </signal>
 <signal name="+18V">
 <contactref element="VD7P" pad="C"/>
+<contactref element="VD2P3" pad="C"/>
+<wire x1="82.07375" y1="-93.345" x2="-401.32" y2="-187.325" width="0" layer="19" extent="1-1"/>
 </signal>
 <signal name="+3V">
@@
 <signal name="-18V">
 <contactref element="VD9P" pad="A"/>
+<contactref element="VD9P1" pad="A"/>
+<wire x1="141.605" y1="-62.70625" x2="-383.54" y2="-225.425" width="0" layer="19" extent="1-1"/>
 </signal>
 <signal name="+6V">
@@
 <signal name="+7V5">
 <contactref element="VD5P" pad="C"/>
+<contactref element="VD2P2" pad="C"/>
+<wire x1="-353.695" y1="82.55" x2="119.6975" y2="-80.48625" width="0" layer="19" extent="1-1"/>
 </signal>
 <signal name="N$107">
@@
 <contactref element="IC5" pad="3"/>
 <contactref element="C2" pad="+"/>
+<contactref element="C3" pad="+"/>
+<wire x1="-376.555" y1="89.4588" x2="-402.59" y2="-179.705" width="0" layer="19" extent="1-1"/>
 <wire x1="-368.935" y1="92.71" x2="-376.555" y2="89.4588" width="0" layer="19" extent="1-1"/>
 </signal>
@@
 <signal name="N$188">
 <contactref element="VD2P1" pad="A"/>
-</signal>
-<signal name="N$187">
-<contactref element="VD2P1" pad="C"/>
-<contactref element="R8P3" pad="2"/>
-<wire x1="-370.525" y1="83.82" x2="-360.68" y2="82.55" width="0" layer="19" extent="1-1"/>
+<contactref element="C2" pad="-"/>
+<contactref element="C3" pad="-"/>
+<wire x1="-366.395" y1="92.71" x2="-400.05" y2="-179.705" width="0" layer="19" extent="1-1"/>
+<wire x1="-360.68" y1="100.33" x2="-366.395" y2="92.71" width="0" layer="19" extent="1-1"/>
 </signal>
 <signal name="N$189">
 <contactref element="R8P2" pad="2"/>
+<contactref element="R8P3" pad="1"/>
 <contactref element="IC5" pad="5"/>
-<contactref element="R8P3" pad="1"/>
-<wire x1="-373.1514" y1="89.4588" x2="-378.78" y2="83.82" width="0" layer="19" extent="1-1"/>
 <wire x1="-372.425" y1="83.82" x2="-378.78" y2="83.82" width="0" layer="19" extent="1-1"/>
+<wire x1="-373.1514" y1="89.4588" x2="-372.425" y2="83.82" width="0" layer="19" extent="1-1"/>
 </signal>
 <signal name="N$190">
-<contactref element="C2" pad="-"/>
 <contactref element="VD2P2" pad="A"/>
-<wire x1="-353.695" y1="100.33" x2="-366.395" y2="92.71" width="0" layer="19" extent="1-1"/>
+</signal>
+<signal name="N$192">
+<contactref element="Q1" pad="3"/>
+</signal>
+<signal name="N$193">
+<contactref element="Q1" pad="2"/>
+</signal>
+<signal name="N$194">
+<contactref element="Q1" pad="1"/>
+</signal>
+<signal name="N$195">
+<contactref element="VD2P3" pad="A"/>
+</signal>
+<signal name="N$196">
+<contactref element="VD10P1" pad="A"/>
 </signal>
 <signal name="N$191">
-<contactref element="VD2P2" pad="C"/>
+<contactref element="VD9P3" pad="C"/>
+</signal>
+<signal name="N$197">
+<contactref element="VD9P1" pad="C"/>
 </signal>
 </signals>

Commit message: .
Parts:
- removed VD2P1: SR5200, diode:CB429-17
- added D16: SBL3040PT, diodes:TO247H
- moved VD10P1 103.4 mm to (-322.6, -118.7)
- moved Q1 33.3 mm to (-368.9, -127.0)
Connections:
- removed net N$188: C2.-, C3.-, VD2P1.A
- new net N$187: C2.-, C3.-, D16.1, D16.3
- net +5VUSB: now also D16.2; no longer VD2P1.C
Changed lines of the file:
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@@
 <element name="R23" library="rcl" package="M0805" value="27" x="-276.225" y="123.19" rot="MR180"/>
 <element name="IC5" library="XL6009" package="TO263-5" value="XL6009" x="-376.555" y="95.25"/>
-<element name="VD2P1" library="diode" package="CB429-17" value="SR5200" x="-360.68" y="91.44" rot="R90"/>
 <element name="C2" library="rcl" package="E2,5-5" value="22m" x="-367.665" y="92.71"/>
 <element name="R8P2" library="rcl" package="M0805" value="1k" x="-379.73" y="83.82"/>
@@
 <element name="T1P1" library="b0f" package="R23X14" value="" x="-370.205" y="117.475"/>
 <element name="VD2P2" library="diode" package="CB429-17" value="SR5200" x="-353.695" y="91.44" rot="R90"/>
-<element name="Q1" library="transistor-fet" package="P-TO247" value="" x="-396.24" y="-146.05"/>
+<element name="Q1" library="transistor-fet" package="P-TO247" value="" x="-368.935" y="-127"/>
 <element name="C3" library="rcl" package="E2,5-5" value="22m" x="-401.32" y="-179.705"/>
 <element name="VD2P3" library="diode" package="CB429-17" value="SR5200" x="-392.43" y="-187.325"/>
-<element name="VD10P1" library="diode" package="CB429-17" value="" x="-392.43" y="-194.945"/>
+<element name="VD10P1" library="diode" package="CB429-17" value="" x="-322.58" y="-118.745"/>
 <element name="VD9P3" library="diode" package="CB429-17" value="" x="-392.43" y="-217.805"/>
 <element name="VD9P1" library="diode" package="CB429-17" value="" x="-392.43" y="-225.425"/>
+<element name="D16" library="diodes" package="TO247H" value="SBL3040PT" x="-337.82" y="86.995"/>
 </elements>
 <signals>
@@
 <contactref element="F_MAIN_POWER" pad="14"/>
 <contactref element="VD10P1" pad="C"/>
+<wire x1="-362.6075" y1="-24.4475" x2="-331.47" y2="-118.745" width="0" layer="19" extent="1-1"/>
+<wire x1="-365.1275" y1="-14.9225" x2="-362.6075" y2="-24.4475" width="0" layer="19" extent="1-1"/>
+<wire x1="-362.2675" y1="5.3975" x2="-365.1275" y2="-14.9225" width="0" layer="19" extent="1-1"/>
+<wire x1="-117.16" y1="-58.42" x2="-331.47" y2="-118.745" width="0" layer="19" extent="1-1"/>
 <wire x1="-39.95" y1="-29.5" x2="-117.16" y2="-58.42" width="0" layer="19" extent="1-1"/>
 <wire x1="-40.27" y1="-26.31" x2="-39.95" y2="-29.5" width="0" layer="19" extent="1-1"/>
@@
 <wire x1="-110.719" y1="57.074" x2="-41.7" y2="-22" width="0" layer="19" extent="1-16"/>
 <wire x1="-140.1" y1="163.71" x2="-111.125" y2="62.865" width="0" layer="19" extent="16-16"/>
-<wire x1="-362.6075" y1="-24.4475" x2="-117.16" y2="-58.42" width="0" layer="19" extent="1-1"/>
-<wire x1="-365.1275" y1="-14.9225" x2="-362.6075" y2="-24.4475" width="0" layer="19" extent="1-1"/>
-<wire x1="-362.2675" y1="5.3975" x2="-365.1275" y2="-14.9225" width="0" layer="19" extent="1-1"/>
-<wire x1="-401.32" y1="-194.945" x2="-362.6075" y2="-24.4475" width="0" layer="19" extent="1-1"/>
 </signal>
 <signal name="N$9">
@@
 <contactref element="VD2P" pad="C"/>
 <contactref element="C7P" pad="+"/>
-<contactref element="VD2P1" pad="C"/>
 <contactref element="R8P3" pad="2"/>
+<contactref element="D16" pad="2"/>
 <wire x1="3.175" y1="-93.98" x2="-29.05375" y2="-90.17" width="0" layer="19" extent="1-1"/>
 <wire x1="35.8775" y1="-96.2025" x2="3.175" y2="-93.98" width="0" layer="19" extent="1-1"/>
-<wire x1="-360.68" y1="82.55" x2="-29.05375" y2="-90.17" width="0" layer="19" extent="1-1"/>
-<wire x1="-370.525" y1="83.82" x2="-360.68" y2="82.55" width="0" layer="19" extent="1-1"/>
+<wire x1="-337.82" y1="79.375" x2="-29.05375" y2="-90.17" width="0" layer="19" extent="1-1"/>
+<wire x1="-370.525" y1="83.82" x2="-337.82" y2="79.375" width="0" layer="19" extent="1-1"/>
 </signal>
 <signal name="+18V">
@@
 <contactref element="IC5" pad="4"/>
 </signal>
-<signal name="N$188">
-<contactref element="VD2P1" pad="A"/>
-<contactref element="C2" pad="-"/>
-<contactref element="C3" pad="-"/>
-<wire x1="-366.395" y1="92.71" x2="-400.05" y2="-179.705" width="0" layer="19" extent="1-1"/>
-<wire x1="-360.68" y1="100.33" x2="-366.395" y2="92.71" width="0" layer="19" extent="1-1"/>
-</signal>
 <signal name="N$189">
 <contactref element="R8P2" pad="2"/>
@@
 <contactref element="VD9P1" pad="C"/>
 </signal>
+<signal name="N$187">
+<contactref element="C2" pad="-"/>
+<contactref element="D16" pad="3"/>
+<contactref element="D16" pad="1"/>
+<contactref element="C3" pad="-"/>
+<wire x1="-343.408" y1="79.375" x2="-332.232" y2="79.375" width="0" layer="19" extent="1-1"/>
+<wire x1="-366.395" y1="92.71" x2="-343.408" y2="79.375" width="0" layer="19" extent="1-1"/>
+<wire x1="-400.05" y1="-179.705" x2="-343.408" y2="79.375" width="0" layer="19" extent="1-1"/>
+</signal>
 </signals>

Commit message: .
Connections:
- new net N$188: IC5.2
- new net N$198: R10P.1
- new net N$199: F_MAIN_POWER.14, F_MAIN_POWER.14A
- net !IGNITION: no longer R10P.1
- net +12V: no longer F_MAIN_POWER.14, F_MAIN_POWER.14A
- net GND: no longer IC5.2
Changed lines of the file:
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@@
 <contactref element="C1" pad="-"/>
 <contactref element="IC5" pad="1"/>
-<contactref element="IC5" pad="2"/>
 <contactref element="R8P2" pad="1"/>
 <wire x1="-144.145" y1="-102.87" x2="-126.05" y2="-127.635" width="0" layer="19" extent="1-1"/>
@@
 <wire x1="-380.68" y1="83.82" x2="-367.3475" y2="-3.4925" width="0" layer="19" extent="1-1"/>
 <wire x1="-379.9586" y1="89.4588" x2="-380.68" y2="83.82" width="0" layer="19" extent="1-1"/>
-<wire x1="-378.2568" y1="89.4588" x2="-379.9586" y2="89.4588" width="0" layer="19" extent="1-1"/>
 </signal>
 <signal name="+12V">
@@
 <contactref element="C3P" pad="1"/>
 <contactref element="R11P" pad="2"/>
-<contactref element="F_MAIN_POWER" pad="14A"/>
-<contactref element="F_MAIN_POWER" pad="14"/>
 <contactref element="VD10P1" pad="C"/>
 <wire x1="-362.6075" y1="-24.4475" x2="-331.47" y2="-118.745" width="0" layer="19" extent="1-1"/>
@@
 <wire x1="-12.065" y1="-53.34" x2="-28.09875" y2="-59.055" width="0" layer="19" extent="1-1"/>
 <wire x1="-10.16" y1="-50.165" x2="-12.065" y2="-53.34" width="0" layer="19" extent="1-1"/>
-<wire x1="-2.54" y1="-45.72" x2="-10.16" y2="-50.165" width="0" layer="19" extent="1-1"/>
-<wire x1="-2.54" y1="-43.18" x2="-2.54" y2="-45.72" width="0" layer="19" extent="1-1"/>
-<wire x1="5.08" y1="-44.45" x2="-2.54" y2="-45.72" width="0" layer="19" extent="1-1"/>
+<wire x1="5.08" y1="-44.45" x2="-10.16" y2="-50.165" width="0" layer="19" extent="1-1"/>
 <wire x1="7.62" y1="-44.45" x2="5.08" y2="-44.45" width="0" layer="19" extent="1-1"/>
 <wire x1="10.16" y1="-44.45" x2="7.62" y2="-44.45" width="0" layer="19" extent="1-1"/>
@@
 </signal>
 <signal name="!IGNITION">
-<contactref element="R10P" pad="1"/>
 <contactref element="F_MAIN_POWER" pad="1A"/>
 <contactref element="F_MAIN_POWER" pad="1"/>
-<wire x1="-35.56" y1="-45.72" x2="-34.925" y2="-53.025" width="0" layer="19" extent="1-1"/>
 <wire x1="-35.56" y1="-43.18" x2="-35.56" y2="-45.72" width="0" layer="19" extent="1-1"/>
 </signal>
@@
 <wire x1="-400.05" y1="-179.705" x2="-343.408" y2="79.375" width="0" layer="19" extent="1-1"/>
 </signal>
+<signal name="N$188">
+<contactref element="IC5" pad="2"/>
+</signal>
+<signal name="N$198">
+<contactref element="R10P" pad="1"/>
+</signal>
+<signal name="N$199">
+<contactref element="F_MAIN_POWER" pad="14A"/>
+<contactref element="F_MAIN_POWER" pad="14"/>
+<wire x1="-2.54" y1="-43.18" x2="-2.54" y2="-45.72" width="0" layer="19" extent="1-1"/>
+</signal>
 </signals>

Commit message: .
Parts:
- removed IC5: XL6009, XL6009:TO263-5
- removed R4P: 10r, rcl:M0805
- added DA1P-: UC3843N, v-reg:DIL08
- DA1P: value UC3843N -> XL6009; device v-reg:DIL08 -> XL6009:TO263-5
- moved DA1P 379.1 mm to (-376.6, 95.2), flipped to the top
- moved VD9P1 344.1 mm to (-217.8, 71.1)
- moved VD9P3 344.1 mm to (-217.8, 78.7)
- moved VD2P3 344.1 mm to (-217.8, 109.2)
- moved C3 242.5 mm to (-349.2, 57.1)
Connections:
- removed net !IGNITION: F_MAIN_POWER.1, F_MAIN_POWER.1A
- removed net N$186: IC5.4
- removed net N$188: IC5.2
- removed net N$198: R10P.1
- new net !RUN: F_MAIN_POWER.1, F_MAIN_POWER.1A, R10P.1
- new net N$200: 1.1, C3P.1, R11P.2, U$22.1, U$38.1
- net +12V: now also DA1P.4; no longer 1.1, C3P.1, R11P.2, U$22.1, U$38.1
- net GND: now also DA1P-.5, DA1P.1; no longer DA1P.5, IC5.1
- net N$108: now also DA1P.2; no longer R4P.1
- net N$185: now also DA1P.3; no longer IC5.3
- net N$189: now also DA1P.5; no longer IC5.5
- net N$20: now also DA1P-.6; no longer DA1P.6
- net N$22: now also DA1P-.3; no longer DA1P.3
- net N$25: now also DA1P-.8; no longer DA1P.8
- net N$26: now also DA1P-.4; no longer DA1P.4
- net N$28: now also DA1P-.2; no longer DA1P.2
- net N$29: now also DA1P-.1; no longer DA1P.1
- net N$30: now also DA1P-.7; no longer DA1P.7, R4P.2
