File: b0_comp.brd (EAGLE design)
At the start: 93 x 70 mm, 294 parts, among them IC1 КР1006ВИ1(NE555), IC3 LM358D, IC4 78L09F, IC6 MEGA8-AI, IC7 74121N, IC8 4030N, IC9 LM324D, T1P T90, -26 MicroMetals Yellow-W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

Commit message: .
Parts:
- removed 10, 11, 12, 13, 14, 15, 16, 17, 18, 19, 20, 5, 6, 7, 8, 9: T_PIN, b0f:PIN1X1
- removed C1: (no value), rcl:E2,5-5
- removed C2, C3: 22m, rcl:E2,5-5
- removed C5P: 1n, rcl:C025-025X050
- removed C6P: 1n, rcl:C0805
- removed C7P: 470m, rcl:E5-10,5
- removed D11: 2Д213А, diode:D-10
- removed D16: SBL3040PT, diodes:TO247H
- removed DA1P-: UC3843N, v-reg:DIL08
- removed R1P: 100k, rcl:M0805
- removed R2P: 29k*, rcl:M0805
- removed R3P: 330, rcl:M0805
- removed R5P: 10r, rcl:M0805
- removed R6P: 0e15 2w, rcl:R1210
- removed R7P, R8P, R8P2: 1k, rcl:M0805
- removed R8P3: 3k, rcl:M0805
- removed R9P: 0, rcl:M0805
- removed T1P: T90, -26 MicroMetals Yellow-White, b0f:R23X14
- removed T1P1: (no value), b0f:R23X14
- removed U$19, U$20, U$21, U$22, U$23, U$24, U$26, U$27, U$28, U$29, U$30, U$31, U$32, U$33, U$34, U$35, U$36, U$38: T_PIN_NONAME, b0f:PIN1X1N
- removed VD10P, VD10P1, VD3P, VD4P, VD5P, VD7P, VD8P, VD9P, VD9P1, VD9P3: (no value), diode:CB429-17
- removed VD2P, VD2P2, VD2P3: SR5200, diode:CB429-17
- removed VT2: PHD45N03, m_transistor:DPACK
- added L1P: (no value), b0f:R23X14
- added R12P: 1k, rcl:M0805
- C2P: value 100n -> 22m; device rcl:C0805 -> rcl:E2,5-5
- C3P: value 220n -> 22m; device rcl:C075-032X103 -> rcl:E2,5-5
- C4P: value 1n -> 470m; device rcl:C0805 -> rcl:E5-10,5
- R11P: value 67r8w -> 3k; device rcl:0207/15 -> rcl:M0805
- VD1P: value LL4148 -> SBL3040PT; device diode:SOD80C -> diodes:TO247H
- moved DA1P 414.9 mm to (3.81, -70.5), turned to 90 degrees
- moved Q1 101.3 mm to (-445.1, -60.3)
- moved C4P 79.8 mm to (35.6, -41.3)
- moved VD1P 66.2 mm to (25.4, -64.1), turned to 270 degrees
- moved C2P 59.9 mm to (23.5, -77.5), turned to 0 degrees
- moved C3P 51.6 mm to (26.7, -82.5), turned to 0 degrees
- moved R11P 46.7 mm to (16.5, -81.9)
- moved 1 44.8 mm to (-6.35, -87.0)
- moved 2 26.4 mm to (-21.6, -62.2)
- moved 4 23.9 mm to (-4.45, -62.9), turned to 0 degrees
- moved 3 6.75 mm to (-0.64, -85.7), turned to 0 degrees
Connections:
- removed net +18V: VD2P3.C, VD7P.C
- removed net +3V: VD3P.C
- removed net +5VUSB: C7P.+, D16.2, R8P3.2, R9P.2, VD2P.C
- removed net +6V: VD4P.C
- removed net +7V5: VD2P2.C, VD5P.C
- removed net -18V: VD9P.A, VD9P1.A
- removed net N$107: 4.1, 5.1, U$26.1, U$27.1, U$28.1, U$29.1, U$30.1, U$31.1, VD3P.A
- removed net N$162: 6.1, 7.1, U$32.1, U$33.1, U$34.1, U$36.1, VD2P.A
- removed net N$163: R8P.2, R9P.1
- removed net N$165: C3P.2, D11.C, R11P.1
- removed net N$168: 20.1, VD10P.A
- removed net N$172: 16.1, 17.1, VD8P.C
- removed net N$175: 10.1, 11.1, VD5P.A
- removed net N$178: 18.1, VD9P.C
- removed net N$180: 14.1, VD7P.A
- removed net N$187: C2.-, C3.-, D16.1, D16.3
- removed net N$190: VD2P2.A
- removed net N$191: VD9P3.C
- removed net N$195: VD2P3.A
- removed net N$196: VD10P1.A
- removed net N$197: VD9P1.C
- removed net N$20: DA1P-.6, R5P.1, VD1P.C
- removed net N$200: 1.1, C3P.1, R11P.2, U$22.1, U$38.1
- removed net N$22: C6P.1, DA1P-.3, R3P.1
- removed net N$23: R3P.2, R6P.2, VT2.S
- removed net N$24: 2.1, D11.A, U$23.1, U$24.1, VT2.D
- removed net N$25: DA1P-.8, R2P.2
- removed net N$26: C5P.1, DA1P-.4, R2P.1
- removed net N$28: C4P.2, DA1P-.2, R1P.1, R7P.2, R8P.1
- removed net N$29: C4P.1, DA1P-.1, R1P.2
- removed net N$30: C1.+, C2P.1, DA1P-.7
- removed net N$64: 8.1, 9.1, U$35.1, VD4P.A
- removed net N$67: 12.1, 13.1
- net +12V: now also 2.1; no longer VD10P.C, VD10P1.C
- net +5V: now also C4P.+, R11P.2, VD1P.2
- net -12V: no longer 19.1, VD8P.A, VD9P3.A
- net GND: now also 4.1, C4P.-, R12P.1; no longer 15.1, 3.1, C1.-, C2P.2, C5P.2, C6P.2, C7P.-, DA1P-.5, R6P.1, R7P.1, R8P2.1, U$19.1, U$20.1, U$21.1
- net N$185: now also 1.1, C2P.+, C3P.+; no longer C2.+, C3.+
- net N$189: now also R11P.1, R12P.2; no longer R8P2.2, R8P3.1
- net N$21: now also 3.1, C2P.-, C3P.-, VD1P.1, VD1P.3; no longer R5P.2, VD1P.A, VT2.G
Routing:
- net N$22: track 20.3 -> 0.00 mm
- net N$26: track 12.9 -> 0.00 mm
- net GND: track 182.7 -> 174.0 mm
- net N$20: track 5.49 -> 0.00 mm
- net N$29: track 5.37 -> 0.00 mm
- net N$28: track 5.37 -> 0.00 mm
- net N$30: track 3.49 -> 0.00 mm
- net N$25: track 2.86 -> 0.00 mm
