File: b0_comp.brd (EAGLE design)
At the start: 93 x 70 mm, 219 parts, among them IC1 КР1006ВИ1(NE555), IC2 4066N, IC3 LM358D, IC4 78L09F, IC6 MEGA8-AI, IC7 74121N, IC8 4030N, IC9 LM324D

Commit message: .
Parts:
- removed LED1: (no value), led:CHIP-LED0603
- removed R1L1: 5506, opto-resistor:R_O
- R1.1: value 470 -> 430
- VT15: value КТ 361 -> КТ 361А1
Connections:
- removed net N$115: LED1.C, R1.1.2, R1.3.2
- removed net N$116: LCD1.20, LCD1.20@
- removed net N$18: LED1.A, VT15.2
- new net BLA: LCD1.19, LCD1.19@, VT15.2
- new net BLK: LCD1.20, LCD1.20@, R1.1.2, R1.3.2
- net +5V: now also JLCD1.M.1, JLCD1.M.2; no longer LCD1.19, LCD1.19@, R1L1.P$1
- net N$29: now also JLCD1.M.3, JLCD1.M.4; no longer R1L1.P$2
Changed lines of the file:
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@@
 <element name="C2L1" library="rcl" package="E2,5-5" value="47m" x="-400.685" y="-97.155"/>
 <element name="IC2" library="40xx" package="DIL14" value="4066N" x="-411.48" y="-195.58"/>
-<element name="R1.1" library="rcl" package="M0805" value="470" x="-429.26" y="-204.47"/>
+<element name="R1.1" library="rcl" package="M0805" value="430" x="-429.26" y="-204.47"/>
 <element name="VT10" library="m_transistor" package="TO92" value="КТ315Г" x="-427.99" y="-211.455"/>
-<element name="R1L1" library="opto-resistor" package="R_O" value="5506" x="-437.515" y="-219.075"/>
 <element name="R1.2" library="rcl" package="M0805" value="910" x="-438.15" y="-224.79"/>
 <element name="R1.3" library="rcl" package="M0805" value="4к7" x="-438.15" y="-231.14"/>
-<element name="VT15" library="m_transistor" package="TO92" value="КТ 361" x="-436.245" y="-238.125"/>
-<element name="LED1" library="led" package="CHIP-LED0603" value="" x="-443.23" y="-241.935"/>
+<element name="VT15" library="m_transistor" package="TO92" value="КТ 361А1" x="-436.245" y="-238.125"/>
 <element name="R3.1" library="rcl" package="M0805" value="2k2" x="-443.23" y="-246.38"/>
 </elements>
@@
 <contactref element="C9P" pad="1"/>
 <contactref element="C8P" pad="+"/>
-<contactref element="R5." pad="2"/>
-<contactref element="LCD1" pad="19@"/>
-<contactref element="LCD1" pad="19"/>
 <contactref element="LCD1" pad="2@"/>
 <contactref element="LCD1" pad="2"/>
@@
 <contactref element="ARDUINO1" pad="VCC@1"/>
 <wire x1="13.22" y1="-29.96" x2="13.22" y2="-32.5" width="1.27" layer="16"/>
+<contactref element="JLCD1.M" pad="1"/>
+<contactref element="JLCD1.M" pad="2"/>
+<contactref element="R5." pad="2"/>
 <contactref element="R6." pad="2"/>
 <contactref element="VT15" pad="1"/>
-<contactref element="R1L1" pad="P$1"/>
 <wire x1="-260.67" y1="13.335" x2="-266.385" y2="13.335" width="0" layer="19" extent="1-1"/>
 <wire x1="-254.955" y1="13.335" x2="-260.67" y2="13.335" width="0" layer="19" extent="1-1"/>
@@
 <wire x1="-19.935" y1="-8.0375" x2="-30.095" y2="-14.3875" width="0" layer="19" extent="1-1"/>
 <wire x1="-19.68" y1="-25.6" x2="-30.095" y2="-14.3875" width="0" layer="19" extent="16-16"/>
-<wire x1="-29.96" y1="-29.96" x2="-19.68" y2="-25.6" width="0" layer="19" extent="16-16"/>
-<wire x1="-29.96" y1="-32.5" x2="-29.96" y2="-29.96" width="0" layer="19" extent="1-1"/>
 <wire x1="4.69" y1="-20.31" x2="-19.68" y2="-25.6" width="0" layer="19" extent="16-16"/>
 <wire x1="6.985" y1="-19.365" x2="4.69" y2="-20.31" width="0" layer="19" extent="16-16"/>
 <wire x1="8.22" y1="-23.99" x2="6.985" y2="-19.365" width="0" layer="19" extent="16-16"/>
 <wire x1="13.22" y1="-29.96" x2="8.22" y2="-23.99" width="0" layer="19" extent="16-16"/>
+<wire x1="-26.035" y1="22.225" x2="-19.935" y2="-8.0375" width="0" layer="19" extent="1-1"/>
+<wire x1="-28.575" y1="22.225" x2="-26.035" y2="22.225" width="0" layer="19" extent="1-1"/>
 <wire x1="48.0488" y1="-21.074" x2="13.22" y2="-29.96" width="0" layer="19" extent="1-1"/>
 <wire x1="56.515" y1="-29.845" x2="48.0488" y2="-21.074" width="0" layer="19" extent="1-1"/>
@@
 <wire x1="-408.625" y1="-84.455" x2="-266.385" y2="13.335" width="0" layer="19" extent="1-1"/>
 <wire x1="-408.625" y1="-97.155" x2="-408.625" y2="-84.455" width="0" layer="19" extent="1-1"/>
-<wire x1="-439.265" y1="-219.075" x2="-408.625" y2="-97.155" width="0" layer="19" extent="1-1"/>
-<wire x1="-438.785" y1="-239.395" x2="-439.265" y2="-219.075" width="0" layer="19" extent="1-1"/>
+<wire x1="-438.785" y1="-239.395" x2="-408.625" y2="-97.155" width="0" layer="19" extent="1-1"/>
 </signal>
 <signal name="N$1">
@@
 <wire x1="-27.94" y1="27.94" x2="-25.4" y2="27.94" width="0" layer="19" extent="1-1"/>
 </signal>
-<signal name="N$116">
+<signal name="BLK">
 <contactref element="LCD1" pad="20"/>
 <contactref element="LCD1" pad="20@"/>
+<contactref element="R1.3" pad="2"/>
+<contactref element="R1.1" pad="2"/>
+<wire x1="-428.31" y1="-204.47" x2="-437.2" y2="-231.14" width="0" layer="19" extent="1-1"/>
+<wire x1="-32.5" y1="-32.5" x2="-428.31" y2="-204.47" width="0" layer="19" extent="1-1"/>
 <wire x1="-32.5" y1="-29.96" x2="-32.5" y2="-32.5" width="0" layer="19" extent="1-1"/>
 </signal>
@@
 <wire x1="-430.21" y1="-204.47" x2="-430.53" y2="-212.725" width="0" layer="19" extent="1-1"/>
 </signal>
-<signal name="N$115">
-<contactref element="R1.3" pad="2"/>
-<contactref element="LED1" pad="C"/>
-<contactref element="R1.1" pad="2"/>
-<wire x1="-437.2" y1="-231.14" x2="-443.23" y2="-241.185" width="0" layer="19" extent="1-1"/>
-<wire x1="-428.31" y1="-204.47" x2="-437.2" y2="-231.14" width="0" layer="19" extent="1-1"/>
-</signal>
 <signal name="N$29">
 <contactref element="VT10" pad="2"/>
-<contactref element="R1L1" pad="P$2"/>
 <contactref element="R1.2" pad="2"/>
 <contactref element="R1.3" pad="1"/>
 <contactref element="R3." pad="1"/>
+<contactref element="JLCD1.M" pad="3"/>
+<contactref element="JLCD1.M" pad="4"/>
 <wire x1="-427.99" y1="-212.725" x2="-410.525" y2="-90.805" width="0" layer="19" extent="1-1"/>
-<wire x1="-435.765" y1="-219.075" x2="-427.99" y2="-212.725" width="0" layer="19" extent="1-1"/>
-<wire x1="-437.2" y1="-224.79" x2="-435.765" y2="-219.075" width="0" layer="19" extent="1-1"/>
+<wire x1="-437.2" y1="-224.79" x2="-427.99" y2="-212.725" width="0" layer="19" extent="1-1"/>
 <wire x1="-439.1" y1="-231.14" x2="-437.2" y2="-224.79" width="0" layer="19" extent="1-1"/>
-</signal>
-<signal name="N$18">
-<contactref element="VT15" pad="2"/>
-<contactref element="LED1" pad="A"/>
-<wire x1="-436.245" y1="-239.395" x2="-443.23" y2="-242.685" width="0" layer="19" extent="1-1"/>
+<wire x1="-23.495" y1="22.225" x2="-410.525" y2="-90.805" width="0" layer="19" extent="1-1"/>
+<wire x1="-20.955" y1="22.225" x2="-23.495" y2="22.225" width="0" layer="19" extent="1-1"/>
 </signal>
 <signal name="N$25">
@@
 <wire x1="-433.705" y1="-239.395" x2="-444.18" y2="-246.38" width="0" layer="19" extent="1-1"/>
 </signal>
+<signal name="BLA">
+<contactref element="LCD1" pad="19@"/>
+<contactref element="LCD1" pad="19"/>
+<contactref element="VT15" pad="2"/>
+<wire x1="-29.96" y1="-32.5" x2="-436.245" y2="-239.395" width="0" layer="19" extent="1-1"/>
+<wire x1="-29.96" y1="-29.96" x2="-29.96" y2="-32.5" width="0" layer="19" extent="1-1"/>
+</signal>
 </signals>

Commit message: .
Parts:
- added C1: (no value), rcl:C0805
- added C2: 100, rcl:C0805
- added C3: 100n, rcl:C0805
- added IC5: TINY13-20SSU, atmel:8S1
- added ISP2: (no value), arduino_jw:CONN-2X03
- added R1, R13, R2, R3, R7, R9: (no value), rcl:R0805
- added R14: 100k, rcl:R0805
- added R1L1: 5506, opto-resistor:R_O
- added VT16, VT17: КТ315Г, m_transistor:TO92
- moved IC2 192.7 mm to (-262.3, -73.7)
- moved R3.1 192.7 mm to (-294.0, -124.5)
- moved VT10 192.7 mm to (-278.8, -89.5)
- moved VT15 192.7 mm to (-287.0, -116.2)
- moved R1.1 192.7 mm to (-280.0, -82.5)
- moved R1.2 192.7 mm to (-288.9, -102.9)
- moved R1.3 192.7 mm to (-288.9, -109.2)
Connections:
- new net N$105: C1.2, R13.1, VT17.1
- new net N$115: R9.2, VT17.2
- new net N$116: C2.2, C3.2
- new net N$124: IC5.3
- new net N$162: C2.1, R14.1
- new net N$163: C3.1, R14.2
- new net N$18: R3.2, VT16.2
- new net N$26: IC5.1, ISP2.5, R1.2
- new net N$67: IC5.5, ISP2.4, R3.1
- new net N$69: IC5.6, ISP2.1, R9.1
- new net N$71: IC5.7, ISP2.3, R1L1.P$1, R2.2
- new net N$72: R7.2
- new net N$98: R7.1, VT16.1
- net +5V: now also C1.1, IC5.8, ISP2.2, R1.1, R13.2, R1L1.P$2
- net GND: now also IC5.4, ISP2.6, R2.1, VT16.3, VT17.3

Commit message: .
Parts:
- IC5: value TINY13-20SSU -> ATtiny13A; device atmel:8S1 -> atmel:DIL08
- R3: value (none) -> 1k
- VT16: value КТ315Г -> 2Т213В
- moved ISP2 45.1 mm to (-222.9, -145.4), turned to 0 degrees
- moved IC5 23.4 mm to (-208.9, -147.3), turned to 270 degrees
Connections:
- net N$26 renamed RES13
- net N$67 renamed MOSI13
- net N$69 renamed MISO13
- net N$71 renamed SCK13
- removed net N$72: R7.2
- net +5V: now also LCD1.19, LCD1.19@
- net BLA: no longer LCD1.19, LCD1.19@
- net BLK: now also R7.2

Commit message: .
Parts:
- removed C2L1: 47m, rcl:E2,5-5
- removed IC6: MEGA8-AI, atmel:TQFP32-08
- removed R1.1: 430, rcl:M0805
- removed R1.2: 910, rcl:M0805
- removed R1.3: 4к7, rcl:M0805
- removed R3., R3.1: 2k2, rcl:M0805
- removed R4.: 47, rcl:M0805
- removed R5., R6.: 10k, rcl:M0805
- removed VT10: КТ315Г, m_transistor:TO92
- removed VT14, VT2: КТ3102Е, m_transistor:TO92
- removed VT15: КТ 361А1, m_transistor:TO92
- R2: value (none) -> 10k
- R7: value (none) -> 68
- VT16: value 2Т213В -> 2Т312В
- moved C2 215.3 mm to (-194.3, -144.1)
- moved C3 215.3 mm to (-194.3, -156.8)
- moved R14 215.3 mm to (-194.3, -150.5)
Connections:
- removed net AVCC: IC6.18
- removed net BLA: VT15.2
- removed net N$114: R1.1.1, VT10.1
- removed net N$20: R5..1, VT14.2, VT2.1
- removed net N$23: C2L1.+, R4..2, VT14.3, VT2.3
- removed net N$24: C2L1.-, R3..2, VT2.2
- removed net N$25: R3.1.2, R6..1, VT14.1
- removed net N$30: R3.1.1, VT15.3
- net +5V: no longer IC6.4, IC6.6, R5..2, R6..2, VT15.1
- net BLK: no longer R1.1.2, R1.3.2
- net GND: no longer IC6.21, IC6.3, IC6.5, R1.2.1, R4..1, VT10.3
- net MISO13: no longer R9.1
- net N$29: no longer R1.2.2, R1.3.1, R3..1, VT10.2

Commit message: .
Parts:
- added R20: 1k, rcl:R0805
- added VT2: BJT_PNP_TO-92_ECB, m_transistor:TO92
Connections:
- new net N$20: R20.2, VT2.3
- new net N$23: R20.1
Changed lines of the file:
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@@
 <element name="R14" library="rcl" package="R0805" value="100k" x="-194.31" y="-150.495"/>
 <element name="C3" library="rcl" package="C0805" value="100n" x="-194.31" y="-156.845"/>
+<element name="VT2" library="m_transistor" package="TO92" value="BJT_PNP_TO-92_ECB" x="-364.49" y="-163.83"/>
+<element name="R20" library="rcl" package="R0805" value="1k" x="-365.76" y="-172.085"/>
 </elements>
 <signals>
@@
 <wire x1="-193.36" y1="-150.495" x2="-195.26" y2="-156.845" width="0" layer="19" extent="1-1"/>
 </signal>
+<signal name="N$20">
+<contactref element="R20" pad="2"/>
+<contactref element="VT2" pad="3"/>
+<wire x1="-361.95" y1="-165.1" x2="-364.81" y2="-172.085" width="0" layer="19" extent="1-1"/>
+</signal>
+<signal name="N$23">
+<contactref element="R20" pad="1"/>
+</signal>
 </signals>

Commit message: .
Parts:
- added C15, C16, C4: 10n, rcl:C0805
- added R21: 10k, rcl:R0805
- added R22, R23, R24: 47k, rcl:R0805
- moved R20 115.8 mm to (-320.7, -65.4)
- moved VT2 110.5 mm to (-333.4, -57.8)
Connections:
- net N$124 renamed !INT4
- new net N$26: C4.1, R22.2, R23.1
- new net N$67: C15.1, R23.2, R24.1
- new net N$69: C16.1, R24.2
- net GND: now also C15.2, C16.2, C4.2, R21.1
- net MISO13: now also R21.2, R22.1
Routing:
- net GND: track 174.0 -> 184.2 mm
- net N$67: track 0.00 -> 5.09 mm
- net N$26: track 0.00 -> 4.77 mm
- net N$25: track 0.00 -> 4.45 mm
- net N$24: track 0.00 -> 4.45 mm
- net N$69: track 0.00 -> 2.54 mm
- net MISO13: track 0.00 -> 2.54 mm
Changed lines of the file:
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@@
 <dimension x1="-311.15" y1="145.415" x2="-260.985" y2="150.495" x3="-286.0675" y3="90.17" textsize="1.778" layer="21" dtype="horizontal"/>
 <dimension x1="-321.31" y1="144.145" x2="-323.215" y2="97.79" x3="-254.635" y3="120.9675" textsize="1.778" layer="21" dtype="vertical"/>
+<wire x1="-62.865" y1="32.385" x2="-60.325" y2="32.385" width="0.4064" layer="21"/>
+<wire x1="-60.325" y1="32.385" x2="-56.515" y2="32.385" width="0.4064" layer="21"/>
+<wire x1="-56.515" y1="32.385" x2="-52.07" y2="32.385" width="0.4064" layer="21"/>
+<wire x1="-52.07" y1="32.385" x2="-49.53" y2="32.385" width="0.4064" layer="21"/>
+<wire x1="-52.07" y1="37.465" x2="-52.07" y2="32.385" width="0.4064" layer="21"/>
+<wire x1="-56.515" y1="37.465" x2="-56.515" y2="32.385" width="0.4064" layer="21"/>
+<wire x1="-60.325" y1="37.465" x2="-60.325" y2="32.385" width="0.4064" layer="21"/>
+<wire x1="-62.865" y1="38.1" x2="-62.865" y2="37.465" width="0.4064" layer="21"/>
+<wire x1="-62.865" y1="37.465" x2="-62.865" y2="32.385" width="0.4064" layer="21"/>
+<wire x1="-62.865" y1="37.465" x2="-52.07" y2="37.465" width="0.4064" layer="21"/>
+<wire x1="-52.07" y1="37.465" x2="-49.53" y2="37.465" width="0.4064" layer="21"/>
+<wire x1="-49.53" y1="37.465" x2="-49.53" y2="29.845" width="0.4064" layer="21"/>
+<wire x1="-49.53" y1="29.845" x2="-62.865" y2="29.845" width="0.4064" layer="21"/>
+<wire x1="-62.865" y1="29.845" x2="-62.865" y2="32.385" width="0.4064" layer="21"/>
 </plain>
 <attributes>
@@
 <element name="R14" library="rcl" package="R0805" value="100k" x="-194.31" y="-150.495"/>
 <element name="C3" library="rcl" package="C0805" value="100n" x="-194.31" y="-156.845"/>
-<element name="VT2" library="m_transistor" package="TO92" value="BJT_PNP_TO-92_ECB" x="-364.49" y="-163.83"/>
-<element name="R20" library="rcl" package="R0805" value="1k" x="-365.76" y="-172.085"/>
+<element name="VT2" library="m_transistor" package="TO92" value="BJT_PNP_TO-92_ECB" x="-333.375" y="-57.785"/>
+<element name="R20" library="rcl" package="R0805" value="1k" x="-320.675" y="-65.405"/>
+<element name="R21" library="rcl" package="R0805" value="10k" x="-61.595" y="32.385" rot="R90"/>
+<element name="R22" library="rcl" package="R0805" value="47k" x="-60.96" y="35.56"/>
+<element name="C4" library="rcl" package="C0805" value="10n" x="-59.055" y="32.385" rot="R270"/>
+<element name="R23" library="rcl" package="R0805" value="47k" x="-56.515" y="35.56"/>
+<element name="R24" library="rcl" package="R0805" value="47k" x="-52.07" y="35.56"/>
+<element name="C15" library="rcl" package="C0805" value="10n" x="-55.245" y="32.385" rot="R270"/>
+<element name="C16" library="rcl" package="C0805" value="10n" x="-51.435" y="32.385" rot="R270"/>
 </elements>
 <signals>
@@
 <contactref element="VT17" pad="3"/>
 <contactref element="ISP2" pad="6"/>
+<contactref element="C16" pad="2"/>
+<contactref element="C15" pad="2"/>
+<contactref element="R21" pad="1"/>
+<contactref element="C4" pad="2"/>
+<wire x1="-61.595" y1="31.435" x2="-59.055" y2="31.435" width="0.4064" layer="1"/>
+<wire x1="-59.055" y1="31.435" x2="-55.245" y2="31.435" width="0.4064" layer="1"/>
+<wire x1="-55.245" y1="31.435" x2="-51.435" y2="31.435" width="0.4064" layer="1"/>
 <wire x1="-185.42" y1="-130.175" x2="-126.05" y2="-127.635" width="0" layer="19" extent="1-1"/>
 <wire x1="-203.2" y1="-130.175" x2="-185.42" y2="-130.175" width="0" layer="19" extent="1-1"/>
@@
 <wire x1="-84.77" y1="3.81" x2="-87.11" y2="7.3" width="0" layer="19" extent="1-1"/>
 <wire x1="-82.55" y1="-20.5" x2="-84.77" y2="3.81" width="0" layer="19" extent="1-1"/>
-<wire x1="-54.5" y1="7.1" x2="-83.5" y2="15.24" width="0" layer="19" extent="1-16"/>
+<wire x1="-61.595" y1="31.435" x2="-83.5" y2="15.24" width="0" layer="19" extent="1-1"/>
+<wire x1="-54.5" y1="7.1" x2="-55.245" y2="31.435" width="0" layer="19" extent="1-16"/>
 <wire x1="-51.5" y1="6.95" x2="-54.5" y2="7.1" width="0" layer="19" extent="16-16"/>
 <wire x1="-35.865" y1="-14.02" x2="-51.5" y2="6.95" width="0" layer="19" extent="16-16"/>
@@
 <contactref element="IC5" pad="6"/>
 <contactref element="ISP2" pad="1"/>
+<contactref element="R21" pad="2"/>
+<contactref element="R22" pad="1"/>
+<wire x1="-61.595" y1="33.335" x2="-61.91" y2="33.335" width="0.4064" layer="1"/>
+<wire x1="-61.91" y1="33.335" x2="-61.91" y2="35.56" width="0.4064" layer="1"/>
 <wire x1="-205.105" y1="-148.59" x2="-222.885" y2="-145.415" width="0" layer="19" extent="1-1"/>
+<wire x1="-61.91" y1="33.335" x2="-205.105" y2="-148.59" width="0" layer="19" extent="1-1"/>
 </signal>
 <signal name="SCK13">
@@
 <contactref element="IC5" pad="7"/>
 <contactref element="ISP2" pad="3"/>
-<wire x1="-205.105" y1="-146.05" x2="-222.885" y2="-147.955" width="0" layer="19" extent="1-1"/>
 <wire x1="-219.71" y1="-135.1" x2="-222.885" y2="-147.955" width="0" layer="19" extent="1-1"/>
 <wire x1="-209.55" y1="-133.67" x2="-219.71" y2="-135.1" width="0" layer="19" extent="1-1"/>
+<wire x1="-205.105" y1="-146.05" x2="-209.55" y2="-133.67" width="0" layer="19" extent="1-1"/>
 </signal>
 <signal name="N$18">
@@
 <wire x1="-178.435" y1="-133.67" x2="-185.42" y2="-132.715" width="0" layer="19" extent="1-1"/>
 </signal>
-<signal name="N$124">
+<signal name="!INT4">
 <contactref element="IC5" pad="3"/>
 </signal>
@@
 <contactref element="R20" pad="2"/>
 <contactref element="VT2" pad="3"/>
-<wire x1="-361.95" y1="-165.1" x2="-364.81" y2="-172.085" width="0" layer="19" extent="1-1"/>
+<wire x1="-319.725" y1="-65.405" x2="-330.835" y2="-59.055" width="0" layer="19" extent="1-1"/>
 </signal>
 <signal name="N$23">
 <contactref element="R20" pad="1"/>
 </signal>
+<signal name="N$26">
+<contactref element="R22" pad="2"/>
+<contactref element="C4" pad="1"/>
+<contactref element="R23" pad="1"/>
+<wire x1="-60.01" y1="35.56" x2="-59.055" y2="35.56" width="0.4064" layer="1"/>
+<wire x1="-59.055" y1="35.56" x2="-57.465" y2="35.56" width="0.4064" layer="1"/>
+<wire x1="-59.055" y1="33.335" x2="-59.055" y2="35.56" width="0.4064" layer="1"/>
+</signal>
+<signal name="N$67">
+<contactref element="R23" pad="2"/>
+<contactref element="R24" pad="1"/>
+<contactref element="C15" pad="1"/>
+<wire x1="-55.565" y1="35.56" x2="-53.02" y2="35.56" width="0.4064" layer="1"/>
+<wire x1="-55.245" y1="33.335" x2="-55.565" y2="33.335" width="0.4064" layer="1"/>
+<wire x1="-55.565" y1="33.335" x2="-55.565" y2="35.56" width="0.4064" layer="1"/>
+</signal>
+<signal name="N$69">
+<contactref element="R24" pad="2"/>
+<contactref element="C16" pad="1"/>
+<wire x1="-51.435" y1="33.335" x2="-51.12" y2="33.335" width="0.4064" layer="1"/>
+<wire x1="-51.12" y1="33.335" x2="-51.12" y2="35.56" width="0.4064" layer="1"/>
+</signal>
+<signal name="N$24">
+<wire x1="-61.595" y1="35.56" x2="-61.595" y2="40.005" width="0.4064" layer="1"/>
+</signal>
+<signal name="N$25">
+<wire x1="-50.8" y1="35.56" x2="-50.8" y2="40.005" width="0.4064" layer="1"/>
+</signal>
 </signals>

Commit message: +t
Parts:
- added IC10: DS1307, ds1307_pcf8583:DIL08
- added IC6: MEGA8-P, atmel:DIL28-3
Connections:
- removed net MOSI: ARDUINO1.D11, ISP1.4, U$1.18
- new net AVCC: IC6.20
- new net ICP: ARDUINO1.D8
- new net N$30: IC6.14
- net +5V: now also IC10.8, IC6.7
- net DB1: now also ARDUINO1.D11, ISP1.4, U$1.18; no longer ARDUINO1.D8
- net GND: now also IC10.4, IC6.22, IC6.8
Changed lines of the file:
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@@
 <element name="C15" library="rcl" package="C0805" value="10n" x="-55.245" y="32.385" rot="R270"/>
 <element name="C16" library="rcl" package="C0805" value="10n" x="-51.435" y="32.385" rot="R270"/>
+<element name="IC6" library="atmel" package="DIL28-3" value="MEGA8-P" x="-346.71" y="-167.64">
+<attribute name="OC_NEWARK" value="unknown" x="-346.71" y="-167.64" size="1.778" layer="27" display="off"/>
+<attribute name="MPN" value="" x="-346.71" y="-167.64" size="1.778" layer="27" display="off"/>
+<attribute name="MF" value="" x="-346.71" y="-167.64" size="1.778" layer="27" display="off"/>
+<attribute name="OC_FARNELL" value="unknown" x="-346.71" y="-167.64" size="1.778" layer="27" display="off"/>
+</element>
+<element name="IC10" library="ds1307_pcf8583" package="DIL08" value="DS1307" x="-338.455" y="-116.84"/>
 </elements>
 <signals>
@@
 <wire x1="-59.055" y1="31.435" x2="-55.245" y2="31.435" width="0.4064" layer="1"/>
 <wire x1="-55.245" y1="31.435" x2="-51.435" y2="31.435" width="0.4064" layer="1"/>
+<contactref element="IC6" pad="8"/>
+<contactref element="IC6" pad="22"/>
+<contactref element="IC10" pad="4"/>
 <wire x1="-185.42" y1="-130.175" x2="-126.05" y2="-127.635" width="0" layer="19" extent="1-1"/>
 <wire x1="-203.2" y1="-130.175" x2="-185.42" y2="-130.175" width="0" layer="19" extent="1-1"/>
@@
 <wire x1="-367.0275" y1="-35.2425" x2="-364.4265" y2="-29.5275" width="0" layer="19" extent="1-1"/>
 <wire x1="-364.4265" y1="-39.0525" x2="-367.0275" y2="-35.2425" width="0" layer="19" extent="1-1"/>
+<wire x1="-347.98" y1="-163.83" x2="-364.4265" y2="-39.0525" width="0" layer="19" extent="1-1"/>
+<wire x1="-345.44" y1="-171.45" x2="-347.98" y2="-163.83" width="0" layer="19" extent="1-1"/>
+<wire x1="-334.645" y1="-120.65" x2="-345.44" y2="-171.45" width="0" layer="19" extent="1-1"/>
 </signal>
 <signal name="+12V">
@@
 <contactref element="ARDUINO1" pad="VCC@1"/>
 <wire x1="13.22" y1="-29.96" x2="13.22" y2="-32.5" width="1.27" layer="16"/>
+<contactref element="IC6" pad="7"/>
+<contactref element="IC10" pad="8"/>
 <wire x1="-260.67" y1="13.335" x2="-266.385" y2="13.335" width="0" layer="19" extent="1-1"/>
 <wire x1="-254.955" y1="13.335" x2="-260.67" y2="13.335" width="0" layer="19" extent="1-1"/>
@@
 <wire x1="-219.71" y1="-131.6" x2="-213.995" y2="-135.57" width="0" layer="19" extent="1-1"/>
 <wire x1="-220.345" y1="-145.415" x2="-213.995" y2="-135.57" width="0" layer="19" extent="1-1"/>
+<wire x1="-347.98" y1="-171.45" x2="-220.345" y2="-145.415" width="0" layer="19" extent="1-1"/>
+<wire x1="-342.265" y1="-113.03" x2="-347.98" y2="-171.45" width="0" layer="19" extent="1-1"/>
 </signal>
 <signal name="N$1">
@@
 <wire x1="0.385" y1="-23.2775" x2="0.52" y2="-29.96" width="0" layer="19" extent="1-1"/>
 </signal>
-<signal name="DB1">
-<contactref element="LCD1" pad="8@"/>
-<contactref element="LCD1" pad="8"/>
-<wire x1="-2.02" y1="-29.96" x2="-2.02" y2="-32.5" width="1.27" layer="16"/>
-<contactref element="ARDUINO1" pad="D8"/>
-<wire x1="-2.155" y1="-23.2775" x2="-2.02" y2="-29.96" width="0" layer="19" extent="1-1"/>
-</signal>
 <signal name="DB2">
 <contactref element="LCD1" pad="9"/>
@@
 <contactref element="U$1" pad="17"/>
 </signal>
-<signal name="MOSI">
+<signal name="DB1">
 <contactref element="U$1" pad="18"/>
 <contactref element="ARDUINO1" pad="D11"/>
 <contactref element="ISP1" pad="4"/>
+<contactref element="LCD1" pad="8@"/>
+<contactref element="LCD1" pad="8"/>
+<wire x1="-2.02" y1="-29.96" x2="-2.02" y2="-32.5" width="1.27" layer="16"/>
 <wire x1="-2.155" y1="-8.0375" x2="-35.865" y2="-11.48" width="0" layer="19" extent="1-1"/>
-<wire x1="48.0488" y1="-19.804" x2="-2.155" y2="-8.0375" width="0" layer="19" extent="1-1"/>
+<wire x1="-2.02" y1="-29.96" x2="-2.155" y2="-8.0375" width="0" layer="19" extent="1-1"/>
+<wire x1="48.0488" y1="-19.804" x2="-2.02" y2="-29.96" width="0" layer="19" extent="1-1"/>
 </signal>
 <signal name="MISO">
@@
 <wire x1="-50.8" y1="35.56" x2="-50.8" y2="40.005" width="0.4064" layer="1"/>
 </signal>
+<signal name="AVCC">
+<contactref element="IC6" pad="20"/>
+</signal>
+<signal name="N$30">
+<contactref element="IC6" pad="14"/>
+</signal>
+<signal name="ICP">
+<contactref element="ARDUINO1" pad="D8"/>
+</signal>
 </signals>
