File: b0_comp.brd (EAGLE design)
At the start: 93 x 70 mm, 229 parts, among them IC1 КР1006ВИ1(NE555), IC10 DS1307, IC2 4066N, IC3 LM358D, IC4 78L09F, IC5 ATtiny13A, IC6 MEGA8-P, IC7 74121N, IC8 4030N, IC9 LM324D

Commit message: .
Parts:
- removed IC10: DS1307, ds1307_pcf8583:DIL08
Connections:
- net +5V: no longer IC10.8
- net GND: no longer IC10.4
Changed lines of the file:
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@@
 <attribute name="OC_FARNELL" value="unknown" x="-346.71" y="-167.64" size="1.778" layer="27" display="off"/>
 </element>
-<element name="IC10" library="ds1307_pcf8583" package="DIL08" value="DS1307" x="-338.455" y="-116.84"/>
 </elements>
 <signals>
@@
 <contactref element="IC6" pad="8"/>
 <contactref element="IC6" pad="22"/>
-<contactref element="IC10" pad="4"/>
 <wire x1="-185.42" y1="-130.175" x2="-126.05" y2="-127.635" width="0" layer="19" extent="1-1"/>
 <wire x1="-203.2" y1="-130.175" x2="-185.42" y2="-130.175" width="0" layer="19" extent="1-1"/>
@@
 <wire x1="-347.98" y1="-163.83" x2="-364.4265" y2="-39.0525" width="0" layer="19" extent="1-1"/>
 <wire x1="-345.44" y1="-171.45" x2="-347.98" y2="-163.83" width="0" layer="19" extent="1-1"/>
-<wire x1="-334.645" y1="-120.65" x2="-345.44" y2="-171.45" width="0" layer="19" extent="1-1"/>
 </signal>
 <signal name="+12V">
@@
 <wire x1="13.22" y1="-29.96" x2="13.22" y2="-32.5" width="1.27" layer="16"/>
 <contactref element="IC6" pad="7"/>
-<contactref element="IC10" pad="8"/>
 <wire x1="-260.67" y1="13.335" x2="-266.385" y2="13.335" width="0" layer="19" extent="1-1"/>
 <wire x1="-254.955" y1="13.335" x2="-260.67" y2="13.335" width="0" layer="19" extent="1-1"/>
@@
 <wire x1="-220.345" y1="-145.415" x2="-213.995" y2="-135.57" width="0" layer="19" extent="1-1"/>
 <wire x1="-347.98" y1="-171.45" x2="-220.345" y2="-145.415" width="0" layer="19" extent="1-1"/>
-<wire x1="-342.265" y1="-113.03" x2="-347.98" y2="-171.45" width="0" layer="19" extent="1-1"/>
 </signal>
 <signal name="N$1">
