File: b0_comp.sch (EAGLE design)
At the start: 173 parts, among them IC1 КР1006ВИ1(NE555), IC10 4011D, IC2 UC3843N, IC3 LM358D, IC4 78L09F, IC5 NE555, IC6 MEGA8-AI, IC7 74121N, IC8 4030N, IC9 LM324D

Commit message: .
Parts:
- removed D11, D12: (no value), diode:DIODE-SOD80C
- added C12: (no value), rcl:CPOL-EUE2.5-5
- added D10, D9: (no value), diode:DIODE-SOD80C
- added JP8: (no value), Разъёмы штырьковые 2.54мм:PINHD-1X1
- added VT8, VT9: КТ315, m_transistor:BJT_NPN_TO-92_ECB
Connections:
- removed net N$147: D12.A, IC9B.-IN, R906.2
- new net N$102: JP8.1, R101*10.2
- new net N$111: IC9B.-IN, R906.2, VT9.C
- net GND: now also C12.-, D10.A, VT8.B, VT9.B
- net N$14: now also D10.C, D9.A
- net N$145: now also VT8.C; no longer D11.A
- net N$146: now also VT8.E; no longer D11.C
- net N$148: now also VT9.E; no longer D12.C
- net N$18: now also D9.C
- net N$33: now also C12.+
Other:
- note added: "+51.1в 8 -51.1в 9 GND 10 +12в 11 (6v) 12 зажигание 13 спидометр 14"
- note added: "1 +51.1в 2 -51.1в 3 GND (rx) 4 +12в (tx) 5 +12в 6 (3v) 7 (поворот)"
- note added: "РША (вид сверху)"
- note added: "Разъем Дг-3-16 / Рп-3-16 вилка"

Commit message: .
Parts:
- removed R, R16, R9: 5506, opto-resistor:R_O
- removed R101: 1, rcl:R-EU_R0805
- added JLCD1.F, JLCD1.M: (no value), Разъёмы штырьковые 2.54мм:PINHD-1X6
- added R1019: 1, rcl:R-EU_R0805
- added R1HUHUH, R2K,: 1k, rcl:R-EU_R0805
- R1, R2: value 1k -> 5506; device rcl:R-EU_R0805 -> opto-resistor:R_O
Connections:
- removed net N$106: R102*.1, R16.2, R9.2
- new net N$109: JLCD1.F.5, JLCD1.F.6, R2.2
- new net N$112: JLCD1.F.3, JLCD1.F.4, R1.2
- new net N$113: JLCD1.F.1, JLCD1.F.2, R1.1, R2.1
- net +12V: now also R1019.2; no longer R101.2
- net +5V: now also R1HUHUH.2, R2K,.2; no longer R.1, R1.2, R2.2
- net BLA: now also R1019.1; no longer R101.1
- net N$105: now also JLCD1.M.1, JLCD1.M.2; no longer R16.1, R9.1
- net N$43: now also R1HUHUH.1; no longer R1.1
- net N$44: now also R2K,.1; no longer R2.1
- net N$69: now also JLCD1.M.3, JLCD1.M.4, JLCD1.M.5, JLCD1.M.6, R102*.1; no longer R.2, VT3.B
Other:
- moved on the sheet: C102, C103, DA1, L101, R102*, R103*, R104*, R105(BL=2V5), R15, VD101, VT3

Commit message: .
Parts:
- added D11, D12: LL4148, diode:DIODE-SOD80C
- added OK1, OK2: PC123, optocoupler:PC817
- added R102*1: *, rcl:R-EU_R0805
- added R13, R9: 12k, rcl:R-EU_R0805
Connections:
- new net N$106: D11.A, OK2.COL, R9.2
- new net N$114: OK1.A, R102*1.2
- new net N$115: OK1.COL, R13.1
- net +12V: now also R13.2, R9.1
- net GND: now also OK1.EMIT, OK2.EMIT
- net N$100: now also D11.C, D12.C
- net N$105: now also OK1.C
- net N$71: now also L101.2; no longer L101.1
- net N$98: now also L101.1, R102*1.1; no longer L101.2
Other:
- note added: "12v 39k 5v 12k"
- moved on the sheet: C102, L101

Commit message: .
Parts:
- removed C102: 10m, rcl:CPOL-EUE2.5-5
- removed C12: (no value), rcl:CPOL-EUE2.5-5
- removed D11: LL4148, diode:DIODE-SOD80C
- removed JP2: (no value), Разъёмы штырьковые 2.54мм:PINHD-1X1
- removed OK2: PC123, optocoupler:PC817
- removed R101*10: 1, rcl:R-EU_M0805
- removed R101*2: 20k, rcl:R-EU_M0805
- removed R101*4: 10k, rcl:R-EU_M0805
- removed R101*7: 5k1, rcl:R-EU_M0805
- removed R101*8: 100k*, rcl:R-EU_M0805
- removed R101*9: 33k, rcl:R-EU_M0805
- removed R102*: 640, rcl:R-EU_R0805
- removed R104*: 1k, rcl:R-EU_R0805
- removed R105(BL=2V5): 10k, rcl:R-EU_R0805
- removed R13, R9: 12k, rcl:R-EU_R0805
- removed R7: 2k2, rcl:R-TRIMM3296W
- added C2L, C4T: 10m, rcl:CPOL-EUE2.5-5
- added C5T: 100n, rcl:C-EUC0805
- added DA4: MC34063TAD, MC34063:MC34063TAD
- added R10T: 33k, rcl:R-EU_M0805
- added R11T: 1M, rcl:R-EU_M0805
- added R12T: 50, rcl:R-EU_M0805
- added R1L0, R2L0, R3L0: 100k, rcl:R-EU_R0805
- added R1T, R8T: 10k, rcl:R-EU_M0805
- added R4L*: 640, rcl:R-EU_R0805
- added R4L0, R7L*: 1k, rcl:R-EU_R0805
- added R5L(BL=2V5): 10k, rcl:R-EU_R0805
- added R5T: 5k1, rcl:R-EU_M0805
- added R6T: 20k, rcl:R-EU_M0805
- added R7T: 2k2, rcl:R-TRIMM3296W
- added R8L: 12k, rcl:R-EU_R0805
- added R9T: 100k*, rcl:R-EU_M0805
- added TIN: (no value), Разъёмы штырьковые 2.54мм:PINHD-1X1
- added U$14: TL432, TL431:TL432
- added VT10: КТ315Б, m_transistor:BJT_NPN_TO-92_CBE
- added VT11: BJT_PNP_TO-92_ECB, m_transistor:BJT_PNP_TO-92_ECB
- C2T: value 100n -> 100n*
- R2T: value 5k1 -> 51k*
- R4T: value 51k -> 51k*
- renumbered C102-1 to C2T, C102-2 to C1T, C102-3 to C6T, C102-4 to C3T, C103 to C3L, D10 to VD2T, D9 to VD1T, IC5 to DA3, R1 to R1L, R101*3 to R2T, R101*5 to R4T, R101*6 to R3T, R1019 to R3L, R103* to R6L*, R2 to R2L
Connections:
- new net N$116: C2L.-, L101.1, LCD1.BLK, R102*1.1, R4L*.2, R5L(BL=2V5).2, R7L*.2
- new net N$117: R3L0.2, VT11.C
- new net N$118: R4L0.1, VT11.B
- new net N$119: R4L0.2, U$14.C
- new net N$120: R1L0.2, VT11.E
- new net N$121: R2L0.1, U$14.A
- new net N$122: R1L0.1, R2L0.2, R3L0.1, U$14.R
- net +12V: now also C2L.+, R8L.2; no longer C102.+, R13.2, R9.1
- net GND: now also C4T.-, C5T.2, OK1.C, R10T.1, R12T.1, VT10.E; no longer C12.-, OK2.EMIT, R101*9.1, R7.A
- net N$100: no longer D11.C
- net N$102: now also C5T.1, R11T.2; no longer R101*10.2
- net N$105: now also JLCD1.M.3, JLCD1.M.4, JLCD1.M.5, JLCD1.M.6, R5L(BL=2V5).1; no longer JLCD1.M.1, JLCD1.M.2, OK1.C, R105(BL=2V5).1
- net N$106: now also R12T.2, R7T.A; no longer D11.A, OK2.COL, R9.2
- net N$114: now also VT10.B; no longer OK1.A
- net N$115: now also D12.A, R8L.1, VT10.C; no longer OK1.COL, R13.1
- net N$12: now also R1T.1, TIN.1; no longer JP2.1
- net N$16: now also R5T.1, R6T.1; no longer R101*2.1, R101*7.1
- net N$17: now also R6T.2; no longer R101*2.2
- net N$18: now also R1T.2, R5T.2; no longer R101*7.2
- net N$31: now also R7T.E, R7T.S, R8T.1; no longer R101*4.1, R7.E, R7.S
- net N$33: now also C4T.+, R8T.2, R9T.2; no longer C12.+, R101*4.2, R101*8.2
- net N$34: now also R10T.2, R11T.1, R9T.1; no longer R101*10.1, R101*8.1, R101*9.2
- net N$69: now also OK1.COL; no longer JLCD1.M.3, JLCD1.M.4, JLCD1.M.5, JLCD1.M.6, R102*.1
- net N$72: now also R7L*.1; no longer R104*.1
- net N$98: now also JLCD1.M.1, JLCD1.M.2, R4L*.1; no longer C102.-, L101.1, LCD1.BLK, R102*.2, R102*1.1, R104*.2, R105(BL=2V5).2
Other:
- note added: "Vт+ = Vref * (1+ R1/R3) Vт- = Vref * (1+ ((R1*R2)/(R1+R2)) * (1/R3) )"
- note added: "Деление с 9 до 2в, не нужно"
- moved on the sheet: D12, JLCD1.M, JP8, OK1, R15, VD101, VT3, VT4

Commit message: .
Parts:
- added L1: 1uµ, rcl:L0204V
- added R1, R13, R7: 1k, rcl:R-EU_0204/5
- added R2, R9: 1k, rcl:R-TRIMM4G/J
- R10T: value 33k -> 1k
- R9T: value 100k* -> 2.125k*
Connections:
- removed net N$18: C6T.1, DA3./RES, DA3.VCC+, IC4.VO, R1T.2, R2T.2, R4T.2, R5T.2, VD1T.C, VT4.C
- new net N$123: C6T.1, IC4.VO
- net +5V: now also DA3./RES, DA3.VCC+, R1T.2, R2T.2, R4T.2, R5T.2, VD1T.C, VT4.C
Other:
- moved on the sheet: JP8, R6T

Commit message: .
Parts:
- removed R5T: 5k1, rcl:R-EU_M0805
- added D9: (no value), diode:ZENER-DIODESMB
- added R14: 5k, rcl:R-TRIMM3059Y
- R12T: value 50 -> 47
- VD1T, VD2T: value (none) -> LL4148
Connections:
- new net N$124: DA1.FB, R14.S
- new net N$18: C3L.1, DA1.TC
- net +5V: no longer R5T.2
- net GND: now also R14.A; no longer DA1.FB
- net N$100: no longer C3L.1, DA1.TC
- net N$114: now also R14.E
- net N$16: no longer R5T.1
Other:
- note added: "К53-4 15мф 15в"
- note added: "Настройка: На вход [pin 2 DA3 NE555] подать 0в. Настроить делитель на 3.4в на выходе к МК"
- moved on the sheet: LCD2

Commit message: ..
Parts:
- added R7T1: 470к, rcl:R-TRIMM3296W
- added VT12: КП302ВМ, m_transistor:JFET-N_TO-72
- C4T: value 10m -> K53-4 15m 15v
- C5T: value 100n -> K53-19 1m
- R6T: value 20k -> 22k
Connections:
- removed net N$33: C4T.+, R8T.2, R9T.2
- new net N$125: R8T.1, VT4.E
- new net N$126: C4T.+, R7T1.E, R7T1.S, R9T.2, VT12.G
- new net N$127: R7T1.A, VT12.S
- net N$16: now also VT12.D
- net N$31: no longer R8T.1, VT4.E
Other:
- note added: "+51.1в 8 (-51.1в) GND 9 GND 10 +12в 11 (6v) 12 зажигание 13 спидометр 14"
- note added: "+51.1в 8 GND 9 I2 10 I1 11 (3v) 12 зажигание 13 спидометр 14"
- note added: "1 +51.1в 2 GND (-51.1в) 3 GND (rx) 4 +12в 5 +12в (tx) 6 (3v) 7 (поворот)"
- note added: "1 +51.1в 2 GND 3 GND 4 +12в 5 +12в 6 (6v) 7 (поворот)"
- note added: "1.19k 121.5k"
- note added: "KT1"
- note added: "rx tx ?"
- note added: "К53-19 (ниобиевый) толстый плюс"
- note removed: "+51.1в 8 -51.1в 9 GND 10 +12в 11 (6v) 12 зажигание 13 спидометр 14"
- note removed: "1 +51.1в 2 -51.1в 3 GND (rx) 4 +12в (tx) 5 +12в 6 (3v) 7 (поворот)"
- moved on the sheet: C4T, C5T, D9, JP8, R10T, R11T, R12T, R8T, R9T

Commit message: .
Parts:
- added JT1, JT2: (no value), jumper:SJ
- added R8T1: 470k, rcl:R-EU_M0805
- D9: device diode:ZENER-DIODESMB -> diode:SCHOTTKY-DIODESMD
- R7T1: value 470к -> 500к
Connections:
- removed net N$126: C4T.+, R7T1.E, R7T1.S, R9T.2, VT12.G
- new net N$128: R7T1.E, R8T1.2
- new net N$130: C4T.+, JT2.1, R7T1.A, R7T1.S, R9T.2, VT12.G
- new net N$33: D9.C, VT12.D
- net GND: now also JT1.2, JT2.2
- net N$127: now also R8T1.1; no longer R7T1.A
- net N$14: now also JT1.1
- net N$16: now also D9.A; no longer VT12.D
Other:
- note added: "Настройка: На вход [pin 2 DA3 NE555] подать 0в. (JT1) Настроить делитель на 3.4в на выходе к МК"
- note removed: "Настройка: На вход [pin 2 DA3 NE555] подать 0в. Настроить делитель на 3.4в на выходе к МК"
- moved on the sheet: C4T, C5T, JP8, R10T, R11T, R7T1, R8T, R9T
