File: b0_comp.sch (EAGLE design)
At the start: 205 parts, among them IC1 КР1006ВИ1(NE555), IC10 4011D, IC2 UC3843N, IC3 LM358D, IC4 78L09F, IC6 MEGA8-AI, IC7 74121N, IC8 4030N, IC9 LM324D

Commit message: .
Parts:
- removed R12T: 47, rcl:R-EU_M0805
- removed R7T1: 500к, rcl:R-TRIMM3296W
- removed R8T1: 470k, rcl:R-EU_M0805
- removed VT12: КП302ВМ, m_transistor:JFET-N_TO-72
- added JT3: (no value), jumper:SJ
- added Q1: 2N5116, transistor-fet:2N5116
- added R7T2: 500к, rcl:R-TRIMM3296W
- added R8T2: 470k, rcl:R-EU_M0805
- added VT1T: КП302ВМ, m_transistor:JFET-N_TO-72
- R11T: value 1M -> 560k
- R7T: value 2k2 -> 100; device rcl:R-TRIMM3296W -> rcl:R-EU_M0805
- R8T: value 10k -> 2k; device rcl:R-EU_M0805 -> rcl:R-TRIMM3296W
Connections:
- removed net N$106: R12T.2, R7T.A
- new net N$126: R7T2.E, R8T2.2
- new net N$129: Q1.G, R7T2.A, R7T2.S
- new net N$131: Q1.S, R8T2.1
- new net N$133: Q1.D
- new net RTC7: DD2.SQW, JT3.2
- net +5V: no longer VT4.C
- net GND: no longer R12T.1
- net N$12: now also JT3.1
- net N$125: no longer R8T.1
- net N$127: now also R7T.1, VT1T.S; no longer R8T1.1, VT12.S
- net N$128: now also R7T.2, R8T.A; no longer R7T1.E, R8T1.2
- net N$130: now also R8T.E, R8T.S, VT1T.G; no longer R7T1.A, R7T1.S, VT12.G
- net N$16: no longer R6T.1
- net N$31: now also VT4.C; no longer R7T.E, R7T.S
- net N$33: now also VT1T.D; no longer VT12.D
Other:
- note added: "100+1.25k=500mka"
- note added: "JT1 off ON ON off"
- note added: "JT2 off off ON off"
- note added: "JT3 off off off ON"
- note added: "Normal Настроить R9T R10T, на R11T ADC 1024 (3.4в) VT1T Сток 500мка 1hz=104ADC=6.066km/h"
- note removed: "KT1"
- moved on the sheet: C4T, C5T, C6T, D9, IC4, JP8, JT2, R10T, R11T, R6T, R9T, VT4

Commit message: .
Parts:
- removed JP8, TIN: (no value), Разъёмы штырьковые 2.54мм:PINHD-1X1
- added TAHO, TAHOIN: (no value), Разъёмы штырьковые 2.54мм:PINHD-1X1
- Q1: value 2N5116 -> КП103
Connections:
- removed net N$102: C5T.1, JP8.1, R11T.2
- removed net N$130: C4T.+, JT2.1, R8T.E, R8T.S, R9T.2, VT1T.G
- removed net N$133: Q1.D
- new net TAHO: ARDUINO1.A0, C5T.1, R11T.2, TAHO.1
- net GND: now also JT2.1; no longer JT2.2
- net N$12: now also TAHOIN.1; no longer TIN.1
- net N$126: now also R8T2.1; no longer R8T2.2
- net N$129: now also D9.C, VT1T.D
- net N$131: now also R8T2.2; no longer R8T2.1
- net N$33: now also C4T.+, JT2.2, Q1.D, R8T.E, R8T.S, R9T.2, VT1T.G; no longer D9.C, VT1T.D
Other:
- note added: "11k 139k"
- note added: "КП302ВМ 100+1.25k=500mka"
- note removed: "100+1.25k=500mka"

Commit message: jf
Parts:
- removed Q1: КП103, transistor-fet:2N5116
- added IN, OUT: (no value), Разъёмы штырьковые 2.54мм:PINHD-1X1
- added JT4: (no value), jumper:SJ
- added T_R12: 100, rcl:R-EU_M0805
- added T_R14A: 2k, rcl:R-TRIMM3296W
- added T_R14B: (no value), rcl:R-TRIMM3296W
- added T_VT1A: КП302ВМ, m_transistor:JFET-N_TO-72
- added T_VT1B, VT1T.2: КП103, transistor-fet:2N5116
- R2T: value 51k* -> 5k1
Connections:
- new net N$102: JT4.1, T_R14B.A, T_VT1A.D, T_VT1B.G
- new net N$106: T_R12.1, T_VT1A.S, T_VT1B.S
- new net N$130: C4T.+, JT2.2, R9T.2, T_R14A.E, T_VT1A.G, T_VT1B.D
- new net N$132: D9.C, JT4.2
- new net N$135: T_R12.2, T_R14A.A, T_R14A.S, T_R14B.E, T_R14B.S
- net N$129: now also VT1T.2.G; no longer D9.C, Q1.G
- net N$131: now also VT1T.2.S; no longer Q1.S
- net N$33: now also VT1T.2.D; no longer C4T.+, JT2.2, Q1.D, R9T.2
Other:
- note added: "JT4 ON ON off ON"
- note added: "для КП302, КП303 T_VT1A and T_R14A OR для КП103 T_VT1B and T_R14B"
- moved on the sheet: C2T, C3T, D9, DA3, R4T, R7T, R7T2, R8T, R8T2, VT1T

Commit message: .
Parts:
- removed IN, OUT: (no value), Разъёмы штырьковые 2.54мм:PINHD-1X1
- removed R7T: 100, rcl:R-EU_M0805
- removed R7T2: 500к, rcl:R-TRIMM3296W
- removed R8T: 2k, rcl:R-TRIMM3296W
- removed R8T2: 470k, rcl:R-EU_M0805
- removed VT1T: КП302ВМ, m_transistor:JFET-N_TO-72
- removed VT1T.2: КП103, transistor-fet:2N5116
Connections:
- removed net N$126: R7T2.E, R8T2.1
- removed net N$127: R7T.1, VT1T.S
- removed net N$128: R7T.2, R8T.A
- removed net N$129: R7T2.A, R7T2.S, VT1T.2.G, VT1T.D
- removed net N$131: R8T2.2, VT1T.2.S
- removed net N$33: R8T.E, R8T.S, VT1T.2.D, VT1T.G
Other:
- note added: "JT3 off off ON"
- note removed: "JT3 off off off ON"
- note removed: "Деление с 9 до 2в, не нужно"
- moved on the sheet: C1T, C2T, C3T, C4T, C5T, D9, DA3, JT1, JT2, JT3, JT4, R10T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

Commit message: ..
Parts:
- T_VT1A: device m_transistor:JFET-N_TO-72 -> m_transistor:JFET-N_TO-72_SDG
- T_VT1B: device transistor-fet:2N5116 -> m_transistor:JFET-P_TO-18V_SGD
Other:
- moved on the sheet: T_VT1B
Changed lines of the file:
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@@
 <grid distance="100" unitdist="mil" unit="mil" style="lines" multiple="1" display="yes" altdistance="0.01" altunitdist="inch" altunit="inch"/>
 <layers>
-<layer number="1" name="Top" color="4" fill="1" visible="yes" active="no"/>
-<layer number="2" name="Route2" color="1" fill="3" visible="yes" active="no"/>
-<layer number="3" name="Route3" color="4" fill="3" visible="yes" active="no"/>
-<layer number="4" name="Route4" color="1" fill="4" visible="yes" active="no"/>
-<layer number="5" name="Route5" color="4" fill="4" visible="yes" active="no"/>
-<layer number="6" name="Route6" color="1" fill="8" visible="yes" active="no"/>
-<layer number="7" name="Route7" color="4" fill="8" visible="yes" active="no"/>
-<layer number="8" name="Route8" color="1" fill="2" visible="yes" active="no"/>
-<layer number="9" name="Route9" color="4" fill="2" visible="yes" active="no"/>
-<layer number="10" name="Route10" color="1" fill="7" visible="yes" active="no"/>
-<layer number="11" name="Route11" color="4" fill="7" visible="yes" active="no"/>
-<layer number="12" name="Route12" color="1" fill="5" visible="yes" active="no"/>
-<layer number="13" name="Route13" color="4" fill="5" visible="yes" active="no"/>
-<layer number="14" name="Route14" color="1" fill="6" visible="yes" active="no"/>
-<layer number="15" name="Route15" color="4" fill="6" visible="yes" active="no"/>
-<layer number="16" name="Bottom" color="1" fill="1" visible="yes" active="no"/>
-<layer number="17" name="Pads" color="2" fill="1" visible="yes" active="no"/>
-<layer number="18" name="Vias" color="2" fill="1" visible="yes" active="no"/>
-<layer number="19" name="Unrouted" color="6" fill="1" visible="yes" active="no"/>
-<layer number="20" name="Dimension" color="15" fill="1" visible="yes" active="no"/>
-<layer number="21" name="tPlace" color="6" fill="1" visible="yes" active="no"/>
-<layer number="22" name="bPlace" color="7" fill="1" visible="yes" active="no"/>
-<layer number="23" name="tOrigins" color="15" fill="1" visible="yes" active="no"/>
-<layer number="24" name="bOrigins" color="15" fill="1" visible="yes" active="no"/>
-<layer number="25" name="tNames" color="7" fill="1" visible="yes" active="no"/>
-<layer number="26" name="bNames" color="7" fill="1" visible="yes" active="no"/>
-<layer number="27" name="tValues" color="7" fill="1" visible="yes" active="no"/>
-<layer number="28" name="bValues" color="7" fill="1" visible="yes" active="no"/>
+<layer number="1" name="Top" color="4" fill="1" visible="no" active="no"/>
+<layer number="2" name="Route2" color="1" fill="3" visible="no" active="no"/>
+<layer number="3" name="Route3" color="4" fill="3" visible="no" active="no"/>
+<layer number="4" name="Route4" color="1" fill="4" visible="no" active="no"/>
+<layer number="5" name="Route5" color="4" fill="4" visible="no" active="no"/>
+<layer number="6" name="Route6" color="1" fill="8" visible="no" active="no"/>
+<layer number="7" name="Route7" color="4" fill="8" visible="no" active="no"/>
+<layer number="8" name="Route8" color="1" fill="2" visible="no" active="no"/>
+<layer number="9" name="Route9" color="4" fill="2" visible="no" active="no"/>
+<layer number="10" name="Route10" color="1" fill="7" visible="no" active="no"/>
+<layer number="11" name="Route11" color="4" fill="7" visible="no" active="no"/>
+<layer number="12" name="Route12" color="1" fill="5" visible="no" active="no"/>
+<layer number="13" name="Route13" color="4" fill="5" visible="no" active="no"/>
+<layer number="14" name="Route14" color="1" fill="6" visible="no" active="no"/>
+<layer number="15" name="Route15" color="4" fill="6" visible="no" active="no"/>
+<layer number="16" name="Bottom" color="1" fill="1" visible="no" active="no"/>
+<layer number="17" name="Pads" color="2" fill="1" visible="no" active="no"/>
+<layer number="18" name="Vias" color="2" fill="1" visible="no" active="no"/>
+<layer number="19" name="Unrouted" color="6" fill="1" visible="no" active="no"/>
+<layer number="20" name="Dimension" color="15" fill="1" visible="no" active="no"/>
+<layer number="21" name="tPlace" color="6" fill="1" visible="no" active="no"/>
+<layer number="22" name="bPlace" color="7" fill="1" visible="no" active="no"/>
+<layer number="23" name="tOrigins" color="15" fill="1" visible="no" active="no"/>
+<layer number="24" name="bOrigins" color="15" fill="1" visible="no" active="no"/>
+<layer number="25" name="tNames" color="7" fill="1" visible="no" active="no"/>
+<layer number="26" name="bNames" color="7" fill="1" visible="no" active="no"/>
+<layer number="27" name="tValues" color="7" fill="1" visible="no" active="no"/>
+<layer number="28" name="bValues" color="7" fill="1" visible="no" active="no"/>
 <layer number="29" name="tStop" color="7" fill="3" visible="no" active="no"/>
 <layer number="30" name="bStop" color="7" fill="6" visible="no" active="no"/>
@@
 <layer number="35" name="tGlue" color="7" fill="4" visible="no" active="no"/>
 <layer number="36" name="bGlue" color="7" fill="5" visible="no" active="no"/>
-<layer number="37" name="tTest" color="7" fill="1" visible="yes" active="no"/>
-<layer number="38" name="bTest" color="7" fill="1" visible="yes" active="no"/>
+<layer number="37" name="tTest" color="7" fill="1" visible="no" active="no"/>
+<layer number="38" name="bTest" color="7" fill="1" visible="no" active="no"/>
 <layer number="39" name="tKeepout" color="4" fill="11" visible="no" active="no"/>
 <layer number="40" name="bKeepout" color="1" fill="11" visible="no" active="no"/>
@@
 <layer number="44" name="Drills" color="7" fill="1" visible="no" active="no"/>
 <layer number="45" name="Holes" color="7" fill="1" visible="no" active="no"/>
-<layer number="46" name="Milling" color="3" fill="1" visible="yes" active="no"/>
-<layer number="47" name="Measures" color="14" fill="1" visible="yes" active="no"/>
-<layer number="48" name="Document" color="7" fill="1" visible="yes" active="no"/>
-<layer number="49" name="Reference" color="7" fill="1" visible="yes" active="no"/>
-<layer number="50" name="dxf" color="7" fill="1" visible="yes" active="no"/>
-<layer number="51" name="tDocu" color="7" fill="1" visible="yes" active="no"/>
-<layer number="52" name="bDocu" color="7" fill="1" visible="yes" active="no"/>
-<layer number="53" name="tGND_GNDA" color="7" fill="9" visible="yes" active="no"/>
-<layer number="54" name="bGND_GNDA" color="1" fill="9" visible="yes" active="no"/>
-<layer number="56" name="wert" color="7" fill="1" visible="yes" active="no"/>
-<layer number="57" name="tCAD" color="7" fill="1" visible="yes" active="no"/>
+<layer number="46" name="Milling" color="3" fill="1" visible="no" active="no"/>
+<layer number="47" name="Measures" color="14" fill="1" visible="no" active="no"/>
+<layer number="48" name="Document" color="7" fill="1" visible="no" active="no"/>
+<layer number="49" name="Reference" color="7" fill="1" visible="no" active="no"/>
+<layer number="50" name="dxf" color="7" fill="1" visible="no" active="no"/>
+<layer number="51" name="tDocu" color="7" fill="1" visible="no" active="no"/>
+<layer number="52" name="bDocu" color="7" fill="1" visible="no" active="no"/>
+<layer number="53" name="tGND_GNDA" color="7" fill="9" visible="no" active="no"/>
+<layer number="54" name="bGND_GNDA" color="1" fill="9" visible="no" active="no"/>
+<layer number="56" name="wert" color="7" fill="1" visible="no" active="no"/>
+<layer number="57" name="tCAD" color="7" fill="1" visible="no" active="no"/>
 <layer number="90" name="Modules" color="13" fill="1" visible="yes" active="yes"/>
 <layer number="91" name="Nets" color="2" fill="1" visible="yes" active="yes"/>
@@
 <part name="U$17" library="Рамка страницы" deviceset="A5_V" device=""/>
 <part name="U$18" library="Рамка страницы" deviceset="A5_V" device=""/>
-<part name="T_VT1A" library="m_transistor" deviceset="JFET-N" device="_TO-72" value="КП302ВМ"/>
+<part name="T_VT1A" library="m_transistor" deviceset="JFET-N" device="_TO-72_SDG" value="КП302ВМ"/>
 <part name="T_R14A" library="rcl" deviceset="R-TRIMM" device="3296W" value="2k"/>
 <part name="T_R14B" library="rcl" deviceset="R-TRIMM" device="3296W"/>
 <part name="T_R12" library="rcl" deviceset="R-EU_" device="M0805" value="100"/>
-<part name="T_VT1B" library="transistor-fet" deviceset="2N5116" device="" value="КП103"/>
+<part name="T_VT1B" library="m_transistor" deviceset="JFET-P" device="_TO-18V_SGD" value="КП103"/>
 <part name="JT4" library="jumper" deviceset="SJ" device=""/>
+<part name="U$16" library="b0f" deviceset="JFET" device=""/>
 </parts>
 <sheets>
@@
 <attribute name="VALUE" x="90.17" y="103.378" size="1.778" layer="96" rot="MR0"/>
 </instance>
-<instance part="T_VT1B" gate="G$1" x="88.9" y="83.82" smashed="yes" rot="R270">
-<attribute name="NAME" x="76.2" y="84.963" size="1.778" layer="95"/>
-<attribute name="VALUE" x="76.2" y="82.55" size="1.778" layer="96"/>
+<instance part="T_VT1B" gate="G$1" x="88.9" y="83.82" smashed="yes" rot="MR270">
+<attribute name="NAME" x="86.36" y="74.803" size="1.778" layer="95" rot="MR0"/>
+<attribute name="VALUE" x="96.52" y="74.93" size="1.778" layer="96" rot="MR0"/>
 </instance>
 <instance part="JT4" gate="1" x="66.04" y="99.06" smashed="yes" rot="R270">
@@
 <attribute name="VALUE" x="62.23" y="101.6" size="1.778" layer="96" rot="R270"/>
 </instance>
+<instance part="U$16" gate="G$1" x="33.02" y="106.68"/>
 </instances>
 <busses>

Commit message: .
Parts:
- R10T: value 1k -> 120k
- R9T: value 2.125k* -> 6.7k*
- T_R12: value 100 -> 100*
- T_R14B: value (none) -> 5k*
- T_VT1B: value КП103 -> КП103Л
Connections:
- net N$102 renamed I_JFET_IN
- net N$106 renamed I_R
- net N$130 renamed I_C_OUT
Other:
- note added: "Normal Настроить R9T R10T, на R11T ADC 1022-1023 (3.4в) VT1T Сток 500мка 1hz=104ADC=6.066km/h"
- note added: "варианты испытания КП302ВМ R4T 52k 100+1.25k=500mka КП103Л R4T 100k =?270mka"
- note removed: "11k 139k"
- note removed: "Normal Настроить R9T R10T, на R11T ADC 1024 (3.4в) VT1T Сток 500мка 1hz=104ADC=6.066km/h"
- note removed: "КП302ВМ 100+1.25k=500mka"
Changed lines of the file:
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@@
 <part name="VT4" library="m_transistor" deviceset="BJT_NPN" device="_TO-92_CBE" value="КТ3102Е"/>
 <part name="R6T" library="rcl" deviceset="R-EU_" device="M0805" value="22k"/>
-<part name="R9T" library="rcl" deviceset="R-EU_" device="M0805" value="2.125k*"/>
-<part name="R10T" library="rcl" deviceset="R-EU_" device="M0805" value="1k"/>
+<part name="R9T" library="rcl" deviceset="R-EU_" device="M0805" value="6.7k*"/>
+<part name="R10T" library="rcl" deviceset="R-EU_" device="M0805" value="120k"/>
 <part name="GND23" library="supply1v" deviceset="GND" device=""/>
 <part name="R11T" library="rcl" deviceset="R-EU_" device="M0805" value="560k"/>
@@
 <part name="T_VT1A" library="m_transistor" deviceset="JFET-N" device="_TO-72_SDG" value="КП302ВМ"/>
 <part name="T_R14A" library="rcl" deviceset="R-TRIMM" device="3296W" value="2k"/>
-<part name="T_R14B" library="rcl" deviceset="R-TRIMM" device="3296W"/>
-<part name="T_R12" library="rcl" deviceset="R-EU_" device="M0805" value="100"/>
-<part name="T_VT1B" library="m_transistor" deviceset="JFET-P" device="_TO-18V_SGD" value="КП103"/>
+<part name="T_R14B" library="rcl" deviceset="R-TRIMM" device="3296W" value="5k*"/>
+<part name="T_R12" library="rcl" deviceset="R-EU_" device="M0805" value="100*"/>
+<part name="T_VT1B" library="m_transistor" deviceset="JFET-P" device="_TO-18V_SGD" value="КП103Л"/>
 <part name="JT4" library="jumper" deviceset="SJ" device=""/>
 <part name="U$16" library="b0f" deviceset="JFET" device=""/>
@@
 <text x="111.76" y="22.86" size="1.778" layer="98">К53-19 (ниобиевый)
 толстый плюс</text>
-<text x="71.12" y="66.04" size="1.778" layer="98">КП302ВМ 100+1.25k=500mka</text>
-<text x="119.38" y="60.96" size="1.778" layer="98">11k
-139k</text>
+<text x="76.2" y="48.26" size="1.778" layer="98">варианты испытания
+КП302ВМ R4T 52k
+100+1.25k=500mka
+КП103Л R4T 100k
+ =?270mka</text>
 <text x="5.08" y="20.32" size="1.778" layer="98" rot="MR180">JT1
 off
@@
 <text x="35.56" y="20.32" size="1.778" layer="98" rot="MR180">
 Normal
-Настроить R9T R10T, на R11T ADC 1024 (3.4в)
+Настроить R9T R10T, на R11T ADC 1022-1023 (3.4в)
 VT1T Сток 500мка
 1hz=104ADC=6.066km/h</text>
@@
 <attribute name="VALUE" x="7.62" y="77.47" size="1.778" layer="96" rot="MR90"/>
 </instance>
-<instance part="R9T" gate="G$1" x="114.3" y="58.42" rot="R90"/>
-<instance part="R10T" gate="G$1" x="114.3" y="43.18" rot="R90"/>
+<instance part="R9T" gate="G$1" x="114.3" y="58.42" smashed="yes" rot="R90">
+<attribute name="NAME" x="115.57" y="57.3786" size="1.778" layer="95"/>
+<attribute name="VALUE" x="115.57" y="55.118" size="1.778" layer="96"/>
+</instance>
+<instance part="R10T" gate="G$1" x="114.3" y="43.18" smashed="yes" rot="R90">
+<attribute name="NAME" x="115.57" y="44.6786" size="1.778" layer="95"/>
+<attribute name="VALUE" x="115.57" y="42.418" size="1.778" layer="96"/>
+</instance>
 <instance part="GND23" gate="1" x="114.3" y="33.02"/>
 <instance part="R11T" gate="G$1" x="121.92" y="50.8"/>
@@
 <instance part="TAHO" gate="G$1" x="129.54" y="73.66" rot="R90"/>
 <instance part="C4T" gate="G$1" x="106.68" y="58.42" smashed="yes" rot="MR0">
-<attribute name="NAME" x="108.077" y="41.1226" size="1.778" layer="95" rot="MR0"/>
-<attribute name="VALUE" x="108.077" y="38.5826" size="1.778" layer="96" rot="MR0"/>
+<attribute name="NAME" x="105.537" y="69.0626" size="1.778" layer="95" rot="MR0"/>
+<attribute name="VALUE" x="105.537" y="66.5226" size="1.778" layer="96" rot="MR0"/>
 </instance>
 <instance part="GND40" gate="1" x="106.68" y="48.26"/>
@@
 </instance>
 <instance part="GND44" gate="1" x="129.54" y="33.02"/>
-<instance part="D9" gate="G$1" x="66.04" y="88.9" rot="R90"/>
+<instance part="D9" gate="G$1" x="66.04" y="88.9" smashed="yes" rot="R90">
+<attribute name="NAME" x="63.246" y="92.075" size="1.778" layer="95" rot="R180"/>
+<attribute name="VALUE" x="69.469" y="86.614" size="1.778" layer="96" rot="R90"/>
+</instance>
 <instance part="JT1" gate="1" x="20.32" y="45.72" smashed="yes" rot="R270">
 <attribute name="NAME" x="17.78" y="45.72" size="1.778" layer="95" rot="R180"/>
@@
 <instance part="T_R14B" gate="G$1" x="106.68" y="99.06" smashed="yes" rot="R180">
 <attribute name="NAME" x="105.41" y="112.649" size="1.778" layer="95" rot="MR0"/>
-<attribute name="VALUE" x="102.87" y="110.49" size="1.778" layer="96" rot="MR0"/>
+<attribute name="VALUE" x="105.41" y="110.49" size="1.778" layer="96" rot="MR0"/>
 </instance>
 <instance part="T_R12" gate="G$1" x="96.52" y="99.06" smashed="yes" rot="R90">
@@
 </instances>
 <busses>
+<bus name="RTC7">
+<segment>
+<wire x1="5.08" y1="58.42" x2="5.08" y2="48.26" width="0.762" layer="92"/>
+</segment>
+</bus>
 </busses>
 <nets>
@@
 <pinref part="JT3" gate="1" pin="2"/>
 <wire x1="12.7" y1="55.88" x2="12.7" y2="53.34" width="0.1524" layer="91"/>
-<wire x1="12.7" y1="53.34" x2="7.62" y2="53.34" width="0.1524" layer="91"/>
+<wire x1="12.7" y1="53.34" x2="5.08" y2="53.34" width="0.1524" layer="91"/>
 <label x="7.62" y="50.8" size="1.778" layer="95"/>
 </segment>
 </net>
-<net name="N$106" class="0">
+<net name="I_R" class="0">
 <segment>
 <pinref part="T_VT1A" gate="Q1" pin="S"/>
@@
 </segment>
 </net>
-<net name="N$102" class="0">
+<net name="I_JFET_IN" class="0">
 <segment>
 <pinref part="T_R14B" gate="G$1" pin="A"/>
@@
 </segment>
 </net>
-<net name="N$130" class="0">
+<net name="I_C_OUT" class="0">
 <segment>
 <pinref part="R9T" gate="G$1" pin="2"/>

Commit message: .
Parts:
- added R16: 10k, rcl:R-EU_R0805
Connections:
- net +5V: now also R16.2
- net RTC7: now also R16.1
Changed lines of the file:
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@@
 <part name="JT4" library="jumper" deviceset="SJ" device=""/>
 <part name="U$16" library="b0f" deviceset="JFET" device=""/>
+<part name="R16" library="rcl" deviceset="R-EU_" device="R0805" value="10k"/>
 </parts>
 <sheets>
@@
 </instance>
 <instance part="R204" gate="G$1" x="53.34" y="33.02" smashed="yes" rot="MR90">
-<attribute name="NAME" x="54.61" y="36.6014" size="1.778" layer="95" rot="MR180"/>
-<attribute name="VALUE" x="54.61" y="33.782" size="1.778" layer="96" rot="MR180"/>
+<attribute name="NAME" x="54.61" y="46.7614" size="1.778" layer="95" rot="MR180"/>
+<attribute name="VALUE" x="54.61" y="43.942" size="1.778" layer="96" rot="MR180"/>
 </instance>
 <instance part="R203" gate="G$1" x="48.26" y="33.02" smashed="yes" rot="MR90">
@@
 <instance part="R14" gate="G$1" x="-12.7" y="160.02"/>
 <instance part="GND45" gate="1" x="-12.7" y="147.32"/>
+<instance part="R16" gate="G$1" x="58.42" y="33.02" smashed="yes" rot="MR90">
+<attribute name="NAME" x="59.69" y="36.6014" size="1.778" layer="95" rot="MR180"/>
+<attribute name="VALUE" x="59.69" y="33.782" size="1.778" layer="96" rot="MR180"/>
+</instance>
 </instances>
 <busses>
@@
 <wire x1="17.78" y1="25.4" x2="17.78" y2="40.64" width="0.1524" layer="91"/>
 <wire x1="17.78" y1="40.64" x2="48.26" y2="40.64" width="0.1524" layer="91"/>
+<pinref part="R16" gate="G$1" pin="2"/>
+<wire x1="58.42" y1="38.1" x2="58.42" y2="40.64" width="0.1524" layer="91"/>
+<wire x1="58.42" y1="40.64" x2="53.34" y2="40.64" width="0.1524" layer="91"/>
+<junction x="53.34" y="40.64"/>
 </segment>
 <segment>
@@
 <segment>
 <pinref part="DD2" gate="G$1" pin="SQW"/>
-<wire x1="43.18" y1="15.24" x2="53.34" y2="15.24" width="0.1524" layer="91"/>
+<wire x1="43.18" y1="15.24" x2="58.42" y2="15.24" width="0.1524" layer="91"/>
 <label x="45.72" y="15.24" size="1.778" layer="95"/>
-</segment>
-</net>
+<pinref part="R16" gate="G$1" pin="1"/>
+<wire x1="58.42" y1="15.24" x2="58.42" y2="27.94" width="0.1524" layer="91"/>
+<junction x="58.42" y="15.24"/>
+</segment>
+</net>
