File: b0_comp.sch (EAGLE design)
At the start: 255 parts, among them IC1 КР1006ВИ1(NE555), IC3 LM358D, IC4 78L09F, IC6 MEGA8-AI, IC7 74121N, IC8 4030N, IC9 LM324D, T1P T, T1P1 T

Commit message: .
Parts:
- removed 17, 18, 19, 20, 21, 22: T_PIN, b0f:T_PIN
- removed D16, D18, D19, D22: (no value), diode:SCHOTTKY-DIODECB429-17
- removed T1P: T, b0f:T
- added D26: (no value), diode:SCHOTTKY-DIODECB429-17
- T1P1: value T -> T90, -26 MicroMetals Yellow-White
Connections:
- net N$179 renamed -18V
- removed net N$107: 19.P$1, D18.A
- removed net N$162: 21.P$1, D19.A
- removed net N$169: D21.C
- removed net N$170: D11.C
- removed net N$174: D22.C
- removed net N$176: D23.C
- removed net N$177: D17.A
- new net +18V: D26.C
- new net N$180: D26.A
- net +3V: now also D21.C; no longer D19.C
- net +6V: now also D11.C; no longer D18.C
- net +7V5: now also D23.C; no longer D16.C
- net -12V: now also D17.A
- net GND: no longer 14.P$1, 15.P$1, 16.P$1, 18.P$1, 20.P$1, 22.P$1
- net N$173: now also VD2P.A; no longer D22.A
- net N$64: no longer VD2P.A
- net N$67: now also 14.P$1, 15.P$1, 16.P$1; no longer 17.P$1, D16.A
Other:
- note added: "10(0.3x1)"
- note added: "12v"
- note added: "14(0.3x1)"
- note added: "27"
- note added: "3(0.6x1)"
- note added: "30(0.3x1)"
- note added: "4(0.6x1)"
- note added: "5(0.6x4)"
- note added: "8(0.6x4)"
- note added: "T90, -26 MicroMetals Yellow-White"
- note removed: "-12vuart"
- note removed: "-15vuart"
- note removed: "3v"
- note removed: "5.1v2.4a 10w 0.6mm x3"
- note removed: "5vusb"
- note removed: "6v"
- note removed: "7.5v0.5a 15w 0.6mm x1"
- note removed: "7.6v"
- moved on the sheet: 11, 12, 13, 14, 15, 16, D11, D17, D20, D21, D23, D24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

Commit message: ..
Parts:
- removed D11, D17, D20, D21, D23, D24, D26: (no value), diode:SCHOTTKY-DIODECB429-17
- removed T1P1: T90, -26 MicroMetals Yellow-White, b0f:T
- added 17, 18, 19, 20: T_PIN, b0f:T_PIN
- added T1P: T90, -26 MicroMetals Yellow-White, b0f:T
- added U$19, U$20, U$21, U$22, U$23, U$24, U$25, U$26, U$27, U$28, U$29, U$30, U$31, U$32, U$33, U$34, U$35, U$36: T_PIN_NONAME, b0f:T_PIN_NONAME
- added VD10P, VD3P, VD4P, VD5P, VD7P, VD8P, VD9P: (no value), diode:SCHOTTKY-DIODECB429-17
Connections:
- removed net N$165: D21.A
- removed net N$166: D11.A
- removed net N$171: D20.C
- removed net N$173: VD2P.A
- new net N$107: 4.P$1, 5.P$1, U$26.TNN1, U$27.TNN1, U$28.TNN1, U$29.TNN1, U$30.TNN1, U$31.TNN1, VD3P.A
- new net N$162: 6.P$1, 7.P$1, U$32.TNN1, U$33.TNN1, U$34.TNN1, U$36.TNN1, VD2P.A
- net +12V: now also U$22.TNN1, U$23.TNN1, VD10P.C; no longer 2.P$1, 3.P$1, 4.P$1, 5.P$1
- net +18V: now also VD7P.C; no longer D26.C
- net +3V: now also VD3P.C; no longer D21.C
- net +6V: now also VD4P.C; no longer D11.C
- net +7V5: now also VD5P.C; no longer D23.C
- net -12V: now also 19.P$1, VD8P.A; no longer D17.A
- net -18V: now also VD9P.A; no longer D24.A
- net GND: now also 15.P$1, 3.P$1, U$19.TNN1, U$20.TNN1, U$21.TNN1
- net N$168: now also 20.P$1, VD10P.A; no longer D20.A
- net N$172: now also 16.P$1, 17.P$1, VD8P.C; no longer D17.C
- net N$175: now also 10.P$1, 11.P$1, VD5P.A; no longer D23.A
- net N$178: now also 18.P$1, VD9P.C; no longer D24.C
- net N$180: now also 14.P$1, VD7P.A; no longer D26.A
- net N$24: now also 2.P$1, U$24.TNN1, U$25.TNN1; no longer 10.P$1, 6.P$1, 7.P$1, 8.P$1, 9.P$1
- net N$64: now also 8.P$1, 9.P$1, U$35.TNN1, VD4P.A; no longer 11.P$1, 12.P$1, 13.P$1
- net N$67: now also 12.P$1, 13.P$1; no longer 14.P$1, 15.P$1, 16.P$1
Other:
- note added: "3(0.6x2)"
- note added: "I 13+12w 0.6mm x3"
- note added: "Бел."
- note added: "Жёлт."
- note added: "Жёлт. 12V"
- note added: "Жёлт. с Син."
- note added: "Зел."
- note added: "Зел.с Син."
- note added: "Красн."
- note added: "Син."
- note removed: "12v"
- note removed: "12vt"
- note removed: "27"
- note removed: "3(0.6x1)"
- note removed: "I 12w 0.6mm x5"
- moved on the sheet: 10, 11, 12, 13, 14, 15, 16, 2, 3, 4, 5, 6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

Commit message: .
Parts:
- removed U$25: T_PIN_NONAME, b0f:T_PIN_NONAME
- added JP1: (no value), Разъёмы штырьковые 2.54мм:PINHD-2X12
- added U$38: T_PIN_NONAME, b0f:T_PIN_NONAME
- R2P: value 59k -> 29k*
- R9P: value 75 -> 0
Connections:
- net +12V: now also U$38.TNN1; no longer U$23.TNN1
- net N$24: now also U$23.TNN1; no longer U$25.TNN1
Other:
- note added: "5.1v"
- note added: "75*"
- moved on the sheet: 19, 20, C1P, T1P, VD10P

Commit message: .
Parts:
- removed JP1: (no value), Разъёмы штырьковые 2.54мм:PINHD-2X12
- added C1: 470m, rcl:CPOL-EUE5-10.5
- added F1: 5A, fuse:FUSESH22,5
- added F_MAIN_POWER: (no value), b0f:PINHD-2X14
- VT1P: value КТ209 -> КТ203; device m_transistor:BJT_PNP_TO-92_ECB -> m_transistor:BJT_PNP_TO18_EBC
Connections:
- new net N$167: F_MAIN_POWER.5, F_MAIN_POWER.6
- new net N$169: F_MAIN_POWER.7, F_MAIN_POWER.8
- new net N$170: F_MAIN_POWER.10, F_MAIN_POWER.9
- new net N$171: F_MAIN_POWER.11, F_MAIN_POWER.12
- new net N$173: F_MAIN_POWER.13, F_MAIN_POWER.14
- new net N$174: F_MAIN_POWER.15, F_MAIN_POWER.16
- new net N$177: F1.2, F_MAIN_POWER.17, F_MAIN_POWER.18, F_MAIN_POWER.19, F_MAIN_POWER.20
- new net N$182: F_MAIN_POWER.27, F_MAIN_POWER.28
- net !IGNITION: now also F_MAIN_POWER.1, F_MAIN_POWER.2
- net +12V: now also F1.1
- net +5VUSB: now also C1.+
- net GND: now also C1.-, F_MAIN_POWER.21, F_MAIN_POWER.22, F_MAIN_POWER.23, F_MAIN_POWER.24, F_MAIN_POWER.3, F_MAIN_POWER.4
- net N$140: now also JP2.14; no longer JP2.13

Commit message: .
Parts:
- VT1P: value КТ203 -> КТ203Б
Changed lines of the file:
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@@
 <grid distance="100" unitdist="mil" unit="mil" style="lines" multiple="1" display="yes" altdistance="0.01" altunitdist="inch" altunit="inch"/>
 <layers>
-<layer number="1" name="Top" color="4" fill="1" visible="yes" active="no"/>
-<layer number="2" name="Route2" color="1" fill="3" visible="yes" active="no"/>
-<layer number="3" name="Route3" color="4" fill="3" visible="yes" active="no"/>
-<layer number="4" name="Route4" color="1" fill="4" visible="yes" active="no"/>
-<layer number="5" name="Route5" color="4" fill="4" visible="yes" active="no"/>
-<layer number="6" name="Route6" color="1" fill="8" visible="yes" active="no"/>
-<layer number="7" name="Route7" color="4" fill="8" visible="yes" active="no"/>
-<layer number="8" name="Route8" color="1" fill="2" visible="yes" active="no"/>
-<layer number="9" name="Route9" color="4" fill="2" visible="yes" active="no"/>
-<layer number="10" name="Route10" color="1" fill="7" visible="yes" active="no"/>
-<layer number="11" name="Route11" color="4" fill="7" visible="yes" active="no"/>
-<layer number="12" name="Route12" color="1" fill="5" visible="yes" active="no"/>
-<layer number="13" name="Route13" color="4" fill="5" visible="yes" active="no"/>
-<layer number="14" name="Route14" color="1" fill="6" visible="yes" active="no"/>
-<layer number="15" name="Route15" color="4" fill="6" visible="yes" active="no"/>
-<layer number="16" name="Bottom" color="1" fill="1" visible="yes" active="no"/>
-<layer number="17" name="Pads" color="2" fill="1" visible="yes" active="no"/>
-<layer number="18" name="Vias" color="2" fill="1" visible="yes" active="no"/>
-<layer number="19" name="Unrouted" color="6" fill="1" visible="yes" active="no"/>
-<layer number="20" name="Dimension" color="15" fill="1" visible="yes" active="no"/>
-<layer number="21" name="tPlace" color="6" fill="1" visible="yes" active="no"/>
-<layer number="22" name="bPlace" color="7" fill="1" visible="yes" active="no"/>
-<layer number="23" name="tOrigins" color="15" fill="1" visible="yes" active="no"/>
-<layer number="24" name="bOrigins" color="15" fill="1" visible="yes" active="no"/>
-<layer number="25" name="tNames" color="7" fill="1" visible="yes" active="no"/>
-<layer number="26" name="bNames" color="7" fill="1" visible="yes" active="no"/>
-<layer number="27" name="tValues" color="7" fill="1" visible="yes" active="no"/>
-<layer number="28" name="bValues" color="7" fill="1" visible="yes" active="no"/>
+<layer number="1" name="Top" color="4" fill="1" visible="no" active="no"/>
+<layer number="2" name="Route2" color="1" fill="3" visible="no" active="no"/>
+<layer number="3" name="Route3" color="4" fill="3" visible="no" active="no"/>
+<layer number="4" name="Route4" color="1" fill="4" visible="no" active="no"/>
+<layer number="5" name="Route5" color="4" fill="4" visible="no" active="no"/>
+<layer number="6" name="Route6" color="1" fill="8" visible="no" active="no"/>
+<layer number="7" name="Route7" color="4" fill="8" visible="no" active="no"/>
+<layer number="8" name="Route8" color="1" fill="2" visible="no" active="no"/>
+<layer number="9" name="Route9" color="4" fill="2" visible="no" active="no"/>
+<layer number="10" name="Route10" color="1" fill="7" visible="no" active="no"/>
+<layer number="11" name="Route11" color="4" fill="7" visible="no" active="no"/>
+<layer number="12" name="Route12" color="1" fill="5" visible="no" active="no"/>
+<layer number="13" name="Route13" color="4" fill="5" visible="no" active="no"/>
+<layer number="14" name="Route14" color="1" fill="6" visible="no" active="no"/>
+<layer number="15" name="Route15" color="4" fill="6" visible="no" active="no"/>
+<layer number="16" name="Bottom" color="1" fill="1" visible="no" active="no"/>
+<layer number="17" name="Pads" color="2" fill="1" visible="no" active="no"/>
+<layer number="18" name="Vias" color="2" fill="1" visible="no" active="no"/>
+<layer number="19" name="Unrouted" color="6" fill="1" visible="no" active="no"/>
+<layer number="20" name="Dimension" color="15" fill="1" visible="no" active="no"/>
+<layer number="21" name="tPlace" color="6" fill="1" visible="no" active="no"/>
+<layer number="22" name="bPlace" color="7" fill="1" visible="no" active="no"/>
+<layer number="23" name="tOrigins" color="15" fill="1" visible="no" active="no"/>
+<layer number="24" name="bOrigins" color="15" fill="1" visible="no" active="no"/>
+<layer number="25" name="tNames" color="7" fill="1" visible="no" active="no"/>
+<layer number="26" name="bNames" color="7" fill="1" visible="no" active="no"/>
+<layer number="27" name="tValues" color="7" fill="1" visible="no" active="no"/>
+<layer number="28" name="bValues" color="7" fill="1" visible="no" active="no"/>
 <layer number="29" name="tStop" color="7" fill="3" visible="no" active="no"/>
 <layer number="30" name="bStop" color="7" fill="6" visible="no" active="no"/>
@@
 <layer number="35" name="tGlue" color="7" fill="4" visible="no" active="no"/>
 <layer number="36" name="bGlue" color="7" fill="5" visible="no" active="no"/>
-<layer number="37" name="tTest" color="7" fill="1" visible="yes" active="no"/>
-<layer number="38" name="bTest" color="7" fill="1" visible="yes" active="no"/>
+<layer number="37" name="tTest" color="7" fill="1" visible="no" active="no"/>
+<layer number="38" name="bTest" color="7" fill="1" visible="no" active="no"/>
 <layer number="39" name="tKeepout" color="4" fill="11" visible="no" active="no"/>
 <layer number="40" name="bKeepout" color="1" fill="11" visible="no" active="no"/>
@@
 <layer number="44" name="Drills" color="7" fill="1" visible="no" active="no"/>
 <layer number="45" name="Holes" color="7" fill="1" visible="no" active="no"/>
-<layer number="46" name="Milling" color="3" fill="1" visible="yes" active="no"/>
-<layer number="47" name="Measures" color="14" fill="1" visible="yes" active="no"/>
-<layer number="48" name="Document" color="7" fill="1" visible="yes" active="no"/>
-<layer number="49" name="Reference" color="7" fill="1" visible="yes" active="no"/>
-<layer number="50" name="dxf" color="7" fill="1" visible="yes" active="no"/>
-<layer number="51" name="tDocu" color="7" fill="1" visible="yes" active="no"/>
-<layer number="52" name="bDocu" color="7" fill="1" visible="yes" active="no"/>
-<layer number="53" name="tGND_GNDA" color="7" fill="9" visible="yes" active="no"/>
-<layer number="54" name="bGND_GNDA" color="1" fill="9" visible="yes" active="no"/>
-<layer number="56" name="wert" color="7" fill="1" visible="yes" active="no"/>
-<layer number="57" name="tCAD" color="7" fill="1" visible="yes" active="no"/>
+<layer number="46" name="Milling" color="3" fill="1" visible="no" active="no"/>
+<layer number="47" name="Measures" color="14" fill="1" visible="no" active="no"/>
+<layer number="48" name="Document" color="7" fill="1" visible="no" active="no"/>
+<layer number="49" name="Reference" color="7" fill="1" visible="no" active="no"/>
+<layer number="50" name="dxf" color="7" fill="1" visible="no" active="no"/>
+<layer number="51" name="tDocu" color="7" fill="1" visible="no" active="no"/>
+<layer number="52" name="bDocu" color="7" fill="1" visible="no" active="no"/>
+<layer number="53" name="tGND_GNDA" color="7" fill="9" visible="no" active="no"/>
+<layer number="54" name="bGND_GNDA" color="1" fill="9" visible="no" active="no"/>
+<layer number="56" name="wert" color="7" fill="1" visible="no" active="no"/>
+<layer number="57" name="tCAD" color="7" fill="1" visible="no" active="no"/>
 <layer number="90" name="Modules" color="13" fill="1" visible="yes" active="yes"/>
 <layer number="91" name="Nets" color="2" fill="1" visible="yes" active="yes"/>
@@
 <part name="JP2" library="Разъёмы штырьковые 2.54мм" deviceset="PINHD-1X14" device=""/>
 <part name="VD2P" library="diode" deviceset="SCHOTTKY-DIODE" device="CB429-17" value="SR5200"/>
-<part name="VT1P" library="m_transistor" deviceset="BJT_PNP" device="_TO18_EBC" value="КТ203"/>
+<part name="VT1P" library="m_transistor" deviceset="BJT_PNP" device="_TO18_EBC" value="КТ203Б"/>
 <part name="R10P" library="rcl" deviceset="R-EU_" device="M0805" value="10k"/>
 <part name="VD1P" library="diode" deviceset="DIODE-" device="SOD80C" value="LL4148"/>
@@
 <instance part="VT1P" gate="G$1" x="35.56" y="83.82" smashed="yes">
 <attribute name="NAME" x="30.48" y="91.44" size="1.778" layer="95"/>
-<attribute name="VALUE" x="30.48" y="88.9" size="1.778" layer="96"/>
+<attribute name="VALUE" x="27.94" y="88.9" size="1.778" layer="96"/>
 </instance>
 <instance part="R10P" gate="G$1" x="25.4" y="83.82"/>
@@
 <pinref part="R10P" gate="G$1" pin="1"/>
 <wire x1="20.32" y1="83.82" x2="2.54" y2="83.82" width="0.1524" layer="91"/>
-<label x="7.62" y="83.82" size="1.778" layer="95"/>
+<label x="5.08" y="142.24" size="1.778" layer="95" rot="R90"/>
 <pinref part="F_MAIN_POWER" gate="A" pin="2"/>
 <pinref part="F_MAIN_POWER" gate="A" pin="1"/>

Commit message: .
Parts:
- added C3P: 220n, rcl:C-EU075-032X103
- added D11: 2Д213А, diode:DIODE-D-10
- added R11P: 67r8w, rcl:R-EU_0207/15
- C5P: device rcl:C-EUC0805 -> rcl:C-EU025-025X050
- VT2: value PHD45N03LTA -> PHD45N03
- renumbered C1 to C7P, C4 to C2P
Connections:
- removed net N$182: F_MAIN_POWER.27, F_MAIN_POWER.28
- new net N$165: C3P.2, D11.C, R11P.1
- net +12V: now also C3P.1, F_MAIN_POWER.27, F_MAIN_POWER.28, R11P.2
- net N$24: now also D11.A
Other:
- moved on the sheet: C4P, R1P

Commit message: .
Parts:
- added C1: (no value), rcl:CPOL-EUE2.5-5
Connections:
- net GND: now also C1.-
- net N$30: now also C1.+
Other:
- moved on the sheet: C1P, R10P, R4P, VT1P
