File: b0_comp.sch (EAGLE design)
At the start: 274 parts, among them IC1 КР1006ВИ1(NE555), IC3 LM358D, IC4 78L09F, IC6 MEGA8-AI, IC7 74121N, IC8 4030N, IC9 LM324D, T1P T90, -26 MicroMetals Yellow-W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

Commit message: .
Parts:
- added DA5: TL494BD, linear:TL494BD
- added DA6: IR2110SPBF, IR2110:IR2110SPBF
- added R20, R3: 10k, rcl:R-EU_0207/12
- added R21, R22, R23: 27, rcl:R-EU_M0805
Connections:
- new net 0V: DA5.+I1, DA5.+I2, DA5.GND, DA6.COM, DA6.VSS, R20.1, R3.1
- new net N$166: DA5.-I1, DA5.-I2, DA5.OUTC, DA5.VREF
- new net N$176: DA5.C1, DA5.C2, DA6.VCC, R21.1
- new net N$179: DA5.E1, DA6.LIN, R20.2
- new net N$181: DA5.E2, DA6.HIN, R3.2
- new net N$182: DA5.VCC, DA6.VDD, R21.2
- new net N$183: DA6.HO, R22.1
- new net N$184: DA6.LO, R23.1
Other:
- note added: "+35..45v -35..45v +12v -12v"
Changed lines of the file:
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@@
 <part name="C1" library="rcl" deviceset="CPOL-EU" device="E2.5-5"/>
 <part name="GND49" library="supply1v" deviceset="GND" device=""/>
+<part name="DA5" library="linear" deviceset="TL494*" device="D" technology="B"/>
+<part name="DA6" library="IR2110" deviceset="IR2110SPBF" device=""/>
+<part name="GND51" library="supply1v" deviceset="0V" device=""/>
+<part name="R3" library="rcl" deviceset="R-EU_" device="0207/12" value="10k"/>
+<part name="R20" library="rcl" deviceset="R-EU_" device="0207/12" value="10k"/>
+<part name="R21" library="rcl" deviceset="R-EU_" device="M0805" value="27"/>
+<part name="R22" library="rcl" deviceset="R-EU_" device="M0805" value="27"/>
+<part name="R23" library="rcl" deviceset="R-EU_" device="M0805" value="27"/>
 </parts>
 <sheets>
@@
 <instance part="GND5" gate="1" x="50.8" y="40.64"/>
 <instance part="R2P" gate="G$1" x="33.02" y="68.58" smashed="yes">
-<attribute name="NAME" x="29.21" y="70.0786" size="1.778" layer="95"/>
-<attribute name="VALUE" x="26.67" y="74.422" size="1.778" layer="96" rot="R180"/>
+<attribute name="NAME" x="26.67" y="70.0786" size="1.778" layer="95"/>
+<attribute name="VALUE" x="41.91" y="71.882" size="1.778" layer="96" rot="R180"/>
 </instance>
 <instance part="C5P" gate="G$1" x="12.7" y="40.64"/>
@@
 </segment>
 </net>
+</nets>
+</sheet>
+<sheet>
+<plain>
+<text x="96.52" y="33.02" size="1.778" layer="98">+35..45v
+-35..45v
++12v
+-12v</text>
+</plain>
+<instances>
+<instance part="DA5" gate="G$1" x="35.56" y="58.42"/>
+<instance part="DA6" gate="A" x="86.36" y="50.8"/>
+<instance part="GND51" gate="1" x="66.04" y="22.86"/>
+<instance part="R3" gate="G$1" x="58.42" y="35.56" smashed="yes" rot="R90">
+<attribute name="NAME" x="57.15" y="26.4414" size="1.778" layer="95" rot="R180"/>
+<attribute name="VALUE" x="57.15" y="23.622" size="1.778" layer="96" rot="R180"/>
+</instance>
+<instance part="R20" gate="G$1" x="63.5" y="35.56" smashed="yes" rot="R90">
+<attribute name="NAME" x="62.23" y="26.4414" size="1.778" layer="95" rot="R180"/>
+<attribute name="VALUE" x="62.23" y="23.622" size="1.778" layer="96" rot="R180"/>
+</instance>
+<instance part="R21" gate="G$1" x="58.42" y="66.04" smashed="yes" rot="R90">
+<attribute name="NAME" x="64.77" y="69.6214" size="1.778" layer="95" rot="R180"/>
+<attribute name="VALUE" x="64.77" y="66.802" size="1.778" layer="96" rot="R180"/>
+</instance>
+<instance part="R22" gate="G$1" x="104.14" y="71.12"/>
+<instance part="R23" gate="G$1" x="104.14" y="53.34"/>
+</instances>
+<busses>
+</busses>
+<nets>
+<net name="N$166" class="0">
+<segment>
+<pinref part="DA5" gate="G$1" pin="VREF"/>
+<wire x1="50.8" y1="68.58" x2="53.34" y2="68.58" width="0.1524" layer="91"/>
+<wire x1="53.34" y1="68.58" x2="53.34" y2="63.5" width="0.1524" layer="91"/>
+<pinref part="DA5" gate="G$1" pin="OUTC"/>
+<wire x1="53.34" y1="63.5" x2="50.8" y2="63.5" width="0.1524" layer="91"/>
+<pinref part="DA5" gate="G$1" pin="-I1"/>
+<wire x1="20.32" y1="68.58" x2="12.7" y2="68.58" width="0.1524" layer="91"/>
+<wire x1="12.7" y1="68.58" x2="12.7" y2="81.28" width="0.1524" layer="91"/>
+<wire x1="12.7" y1="81.28" x2="53.34" y2="81.28" width="0.1524" layer="91"/>
+<wire x1="53.34" y1="81.28" x2="53.34" y2="68.58" width="0.1524" layer="91"/>
+<pinref part="DA5" gate="G$1" pin="-I2"/>
+<wire x1="20.32" y1="58.42" x2="12.7" y2="58.42" width="0.1524" layer="91"/>
+<wire x1="12.7" y1="58.42" x2="12.7" y2="68.58" width="0.1524" layer="91"/>
+<junction x="12.7" y="68.58"/>
+<junction x="53.34" y="68.58"/>
+</segment>
+</net>
+<net name="0V" class="0">
+<segment>
+<pinref part="DA6" gate="A" pin="COM"/>
+<wire x1="68.58" y1="30.48" x2="66.04" y2="30.48" width="0.1524" layer="91"/>
+<pinref part="GND51" gate="1" pin="0V"/>
+<wire x1="66.04" y1="30.48" x2="66.04" y2="27.94" width="0.1524" layer="91"/>
+<pinref part="DA6" gate="A" pin="VSS"/>
+<wire x1="66.04" y1="27.94" x2="66.04" y2="25.4" width="0.1524" layer="91"/>
+<wire x1="68.58" y1="27.94" x2="66.04" y2="27.94" width="0.1524" layer="91"/>
+<junction x="66.04" y="27.94"/>
+<pinref part="R3" gate="G$1" pin="1"/>
+<wire x1="58.42" y1="30.48" x2="58.42" y2="27.94" width="0.1524" layer="91"/>
+<wire x1="63.5" y1="27.94" x2="66.04" y2="27.94" width="0.1524" layer="91"/>
+<pinref part="R20" gate="G$1" pin="1"/>
+<wire x1="63.5" y1="27.94" x2="63.5" y2="30.48" width="0.1524" layer="91"/>
+<pinref part="DA5" gate="G$1" pin="GND"/>
+<wire x1="50.8" y1="38.1" x2="53.34" y2="38.1" width="0.1524" layer="91"/>
+<wire x1="53.34" y1="38.1" x2="53.34" y2="27.94" width="0.1524" layer="91"/>
+<wire x1="63.5" y1="27.94" x2="58.42" y2="27.94" width="0.1524" layer="91"/>
+<junction x="63.5" y="27.94"/>
+<junction x="58.42" y="27.94"/>
+<wire x1="58.42" y1="27.94" x2="53.34" y2="27.94" width="0.1524" layer="91"/>
+<pinref part="DA5" gate="G$1" pin="+I1"/>
+<wire x1="17.78" y1="73.66" x2="20.32" y2="73.66" width="0.1524" layer="91"/>
+<pinref part="DA5" gate="G$1" pin="+I2"/>
+<wire x1="17.78" y1="63.5" x2="20.32" y2="63.5" width="0.1524" layer="91"/>
+<wire x1="17.78" y1="73.66" x2="17.78" y2="63.5" width="0.1524" layer="91"/>
+<wire x1="17.78" y1="63.5" x2="17.78" y2="27.94" width="0.1524" layer="91"/>
+<wire x1="17.78" y1="27.94" x2="53.34" y2="27.94" width="0.1524" layer="91"/>
+<junction x="17.78" y="63.5"/>
+<junction x="53.34" y="27.94"/>
+</segment>
+</net>
+<net name="N$176" class="0">
+<segment>
+<pinref part="DA5" gate="G$1" pin="C2"/>
+<wire x1="50.8" y1="48.26" x2="53.34" y2="48.26" width="0.1524" layer="91"/>
+<wire x1="53.34" y1="48.26" x2="53.34" y2="58.42" width="0.1524" layer="91"/>
+<pinref part="DA5" gate="G$1" pin="C1"/>
+<wire x1="53.34" y1="58.42" x2="50.8" y2="58.42" width="0.1524" layer="91"/>
+<wire x1="53.34" y1="58.42" x2="58.42" y2="58.42" width="0.1524" layer="91"/>
+<wire x1="58.42" y1="58.42" x2="66.04" y2="58.42" width="0.1524" layer="91"/>
+<wire x1="66.04" y1="58.42" x2="66.04" y2="68.58" width="0.1524" layer="91"/>
+<pinref part="DA6" gate="A" pin="VCC"/>
+<wire x1="66.04" y1="68.58" x2="68.58" y2="68.58" width="0.1524" layer="91"/>
+<junction x="53.34" y="58.42"/>
+<junction x="58.42" y="58.42"/>
+<pinref part="R21" gate="G$1" pin="1"/>
+<wire x1="58.42" y1="60.96" x2="58.42" y2="58.42" width="0.1524" layer="91"/>
+</segment>
+</net>
+<net name="N$179" class="0">
+<segment>
+<pinref part="DA5" gate="G$1" pin="E1"/>
+<wire x1="50.8" y1="53.34" x2="63.5" y2="53.34" width="0.1524" layer="91"/>
+<pinref part="DA6" gate="A" pin="LIN"/>
+<pinref part="R20" gate="G$1" pin="2"/>
+<wire x1="63.5" y1="40.64" x2="63.5" y2="53.34" width="0.1524" layer="91"/>
+<junction x="63.5" y="53.34"/>
+<wire x1="63.5" y1="53.34" x2="68.58" y2="53.34" width="0.1524" layer="91"/>
+</segment>
+</net>
+<net name="N$181" class="0">
+<segment>
+<pinref part="DA5" gate="G$1" pin="E2"/>
+<wire x1="50.8" y1="43.18" x2="58.42" y2="43.18" width="0.1524" layer="91"/>
+<wire x1="58.42" y1="40.64" x2="58.42" y2="43.18" width="0.1524" layer="91"/>
+<pinref part="R3" gate="G$1" pin="2"/>
+<wire x1="58.42" y1="43.18" x2="58.42" y2="55.88" width="0.1524" layer="91"/>
+<junction x="58.42" y="43.18"/>
+<pinref part="DA6" gate="A" pin="HIN"/>
+<wire x1="58.42" y1="55.88" x2="68.58" y2="55.88" width="0.1524" layer="91"/>
+</segment>
+</net>
+<net name="N$182" class="0">
+<segment>
+<pinref part="DA5" gate="G$1" pin="VCC"/>
+<pinref part="DA6" gate="A" pin="VDD"/>
+<wire x1="50.8" y1="73.66" x2="58.42" y2="73.66" width="0.1524" layer="91"/>
+<junction x="58.42" y="73.66"/>
+<pinref part="R21" gate="G$1" pin="2"/>
+<wire x1="58.42" y1="71.12" x2="58.42" y2="73.66" width="0.1524" layer="91"/>
+<wire x1="58.42" y1="73.66" x2="68.58" y2="73.66" width="0.1524" layer="91"/>
+</segment>
+</net>
+<net name="N$183" class="0">
+<segment>
+<pinref part="DA6" gate="A" pin="HO"/>
+<pinref part="R22" gate="G$1" pin="1"/>
+<wire x1="96.52" y1="71.12" x2="99.06" y2="71.12" width="0.1524" layer="91"/>
+</segment>
+</net>
+<net name="N$184" class="0">
+<segment>
+<pinref part="DA6" gate="A" pin="LO"/>
+<pinref part="R23" gate="G$1" pin="1"/>
+<wire x1="96.52" y1="53.34" x2="99.06" y2="53.34" width="0.1524" layer="91"/>
+</segment>
+</net>
